File: pcb/discovery.sch (KiCad schematic (older format))
At the start: 2 parts, among them U1 STM32F4-DISCOVERY, U5 FT230X

Commit message: Added LCD and started wiring busses
Parts:
- added J1: ITDB_TFT, symbol ITDB_TFT
Connections:
- net labels added: LCD_D[0..15], SPI1_CLK, SPI1_MISO, SPI1_MOSI, SPI2_CLK, SPI2_MISO, SPI2_MOSI, USB_D+, USB_D-
- wire segments 25 -> 182
Other:
- moved on the sheet: U5

Commit message: Broke up schematic in a more modular fashion -- Added LCD footprint
Parts:
- removed J1: ITDB_TFT, symbol ITDB_TFT
- added C32: 10n(25V), symbol CAP
- added U8: LSM330DLC, symbol LSM330DLC
Connections:
- net labels added: AUDIO_IN_L, AUDIO_IN_R, LCD_D0, LCD_D1, LCD_D10, LCD_D11, LCD_D12, LCD_D13, LCD_D14, LCD_D15, LCD_D2, LCD_D3, LCD_D4, LCD_D5, LCD_D6, LCD_D7, LCD_D8, LCD_D9, RF_RESET, SPI1_IRQ_RF, SPI1_nCS_LSMa, SPI1_nCS_LSMg, SPI1_nCS_RF
- wire segments 182 -> 159

Commit message: Connected the power pins to some free GPIOs
Connections:
- net labels added: POW_HPWR, POW_MODE, POW_nCHARG, POW_nCHRG
- wire segments 159 -> 165

Commit message: Added external interrupts to for the gyro and acc
Connections:
- net labels added: DEN_G, DRDYg/INT2_G, INT1_A, INT1_G, INT2_A
- wire segments 165 -> 174

Commit message: Added interrupt channel for RF to EXTI1
Connections:
- wire segments 174 -> 175

Commit message: Hardly anything
Connections:
- wire segments 175 -> 176

Commit message: Rearranged the external interrupt pins. Changed the name of the RF IRQ line net.
Connections:
- net labels added: SPI_IRQ_RF
- net labels removed: SPI1_IRQ_RF
Changed lines of the file:
@@
-EESchema Schematic File Version 2  date Thu 06 Sep 2012 03:52:35 PM EDT
+EESchema Schematic File Version 2  date 9/7/2012 11:59:32 AM
 LIBS:power
 LIBS:device
@@
 Sheet 3 6
 Title ""
-Date "6 sep 2012"
+Date "7 sep 2012"
 Rev ""
 Comp ""
@@
 $EndDescr
 Wire Wire Line
-	4850 3550 5100 3550
+	1350 3750 1200 3750
+Wire Wire Line
+	3600 4050 3450 4050
 Wire Wire Line
 	7700 1600 8000 1600
-Wire Wire Line
-	7000 3650 7200 3650
 Wire Wire Line
 	7000 3750 7200 3750
@@
 	7000 4050 7200 4050
 Wire Wire Line
-	1350 3750 1200 3750
-Text Label 1200 3750 2    40   ~ 0
-SPI1_IRQ_RF
+	3450 3950 3600 3950
+Text Label 3600 3950 0    40   ~ 0
+SPI_IRQ_RF
 Text Label 7200 4050 0    40   ~ 0
 DEN_G
@@
 Text Label 8000 1500 0    40   ~ 0
 DRDYg/INT2_G
-Text Label 4850 3550 2    40   ~ 0
+Text Label 3600 4050 0    40   ~ 0
 DRDYg/INT2_G
 Text Label 8000 1400 0    40   ~ 0
@@
 Text Label 4850 3650 2    40   ~ 0
 INT2_A
-Text Label 7200 3650 0    40   ~ 0
+Text Label 1200 3750 2    40   ~ 0
 INT1_G
 Text HLabel 10150 2350 2    60   Input ~ 0
@@
 LCD_D[0..15]
 Text HLabel 10150 1250 2    60   Input ~ 0
-SPI1_IRQ_RF
+SPI_IRQ_RF
 Text HLabel 10150 1150 2    60   Output ~ 0
 SPI1_nCS_RF
@@
 SPI1_MISO
 Text Label 9350 1250 2    60   ~ 0
-SPI1_IRQ_RF
+SPI_IRQ_RF
 Text Label 9350 1150 2    60   ~ 0
 SPI1_nCS_RF
