File: pcb/discovery.sch (KiCad schematic (older format))
At the start: 4 parts, among them U1 STM32F4-DISCOVERY, U5 FT230X, U8 LSM330DLC

Commit message: Added Swtiches as well as associated them to the appropriate external interrupts
Parts:
- added R21, R22, R23, R24, R25: 10k, symbol RES
- added S1, S2, S3, S4, S5: EVQ-Q2S03W, symbol EVQ-Q2S03W
Connections:
- wire segments 176 -> 187
Changed lines of the file:
@@
-EESchema Schematic File Version 2  date 9/7/2012 11:59:32 AM
+EESchema Schematic File Version 2  date 9/7/2012 2:41:25 PM
 LIBS:power
 LIBS:device
@@
 $EndDescr
 Wire Wire Line
+	8875 4075 8550 4075
+Connection ~ 8700 4075
+Wire Wire Line
+	8550 5225 8700 5225
+Wire Wire Line
+	8700 5225 8700 2925
+Wire Wire Line
+	8700 2925 8550 2925
+Wire Wire Line
+	8250 4825 8400 4825
+Wire Wire Line
+	8250 4275 8400 4275
+Wire Wire Line
 	1350 3750 1200 3750
 Wire Wire Line
@@
 Wire Wire Line
 	3450 3950 3600 3950
+Wire Wire Line
+	8250 3125 8400 3125
+Wire Wire Line
+	8250 3725 8400 3725
+Wire Wire Line
+	8400 5425 8250 5425
+Wire Wire Line
+	8550 4625 8700 4625
+Connection ~ 8700 4625
+Wire Wire Line
+	8550 3525 8700 3525
+Connection ~ 8700 3525
+Text GLabel 8875 4075 2    60   Input ~ 0
+Vreg
+$Comp
+L RES R25
+U 1 1 504A3CA8
+P 8400 5225
+F 0 "R25" H 8470 5190 50  0000 L TNN
+F 1 "10k" H 8400 5280 30  0000 C BNN
+	1    8400 5225
+	1    0    0    -1
+$EndComp
+$Comp
+L RES R24
+U 1 1 504A3CA3
+P 8400 4625
+F 0 "R24" H 8470 4590 50  0000 L TNN
+F 1 "10k" H 8400 4680 30  0000 C BNN
+	1    8400 4625
+	1    0    0    -1
+$EndComp
+$Comp
+L RES R23
+U 1 1 504A3CA0
+P 8400 4075
+F 0 "R23" H 8470 4040 50  0000 L TNN
+F 1 "10k" H 8400 4130 30  0000 C BNN
+	1    8400 4075
+	1    0    0    -1
+$EndComp
+$Comp
+L RES R22
+U 1 1 504A3C9C
+P 8400 3525
+F 0 "R22" H 8470 3490 50  0000 L TNN
+F 1 "10k" H 8400 3580 30  0000 C BNN
+	1    8400 3525
+	1    0    0    -1
+$EndComp
+$Comp
+L RES R21
+U 1 1 504A3C92
+P 8400 2925
+F 0 "R21" H 8470 2890 50  0000 L TNN
+F 1 "10k" H 8400 2980 30  0000 C BNN
+	1    8400 2925
+	1    0    0    -1
+$EndComp
+$Comp
+L GND #PWR?
+U 1 1 504A3C7D
+P 8400 5425
+F 0 "#PWR?" H 8400 5425 30  0001 C CNN
+F 1 "GND" H 8400 5355 30  0001 C CNN
+	1    8400 5425
+	0    -1   1    0
+$EndComp
+$Comp
+L GND #PWR?
+U 1 1 504A3C49
+P 8400 4825
+F 0 "#PWR?" H 8400 4825 30  0001 C CNN
+F 1 "GND" H 8400 4755 30  0001 C CNN
+	1    8400 4825
+	0    -1   1    0
+$EndComp
+$Comp
+L GND #PWR?
+U 1 1 504A3C3E
+P 8400 3725
+F 0 "#PWR?" H 8400 3725 30  0001 C CNN
+F 1 "GND" H 8400 3655 30  0001 C CNN
+	1    8400 3725
+	0    -1   1    0
+$EndComp
+$Comp
+L GND #PWR?
+U 1 1 504A3BFE
+P 8400 4275
+F 0 "#PWR?" H 8400 4275 30  0001 C CNN
+F 1 "GND" H 8400 4205 30  0001 C CNN
+	1    8400 4275
+	0    -1   1    0
+$EndComp
+$Comp
+L GND #PWR?
+U 1 1 504A3BF9
+P 8400 3125
+F 0 "#PWR?" H 8400 3125 30  0001 C CNN
+F 1 "GND" H 8400 3055 30  0001 C CNN
+	1    8400 3125
+	0    -1   1    0
+$EndComp
+$Comp
+L EVQ-Q2S03W S5
+U 1 1 504A3774
+P 8075 5325
+F 0 "S5" H 8075 5150 60  0000 C CNN
+F 1 "EVQ-Q2S03W" H 8075 5525 60  0000 C CNN
+	1    8075 5325
+	1    0    0    -1
+$EndComp
+$Comp
+L EVQ-Q2S03W S4
+U 1 1 504A376D
+P 8075 4725
+F 0 "S4" H 8075 4550 60  0000 C CNN
+F 1 "EVQ-Q2S03W" H 8075 4950 60  0000 C CNN
+	1    8075 4725
+	1    0    0    -1
+$EndComp
+$Comp
+L EVQ-Q2S03W S3
+U 1 1 504A3765
+P 8075 4175
+F 0 "S3" H 8075 4000 60  0000 C CNN
+F 1 "EVQ-Q2S03W" H 8075 4375 60  0000 C CNN
+	1    8075 4175
+	1    0    0    -1
+$EndComp
+$Comp
+L EVQ-Q2S03W S2
+U 1 1 504A375D
+P 8075 3625
+F 0 "S2" H 8075 3450 60  0000 C CNN
+F 1 "EVQ-Q2S03W" H 8075 3825 60  0000 C CNN
+	1    8075 3625
+	1    0    0    -1
+$EndComp
+$Comp
+L EVQ-Q2S03W S1
+U 1 1 504A3753
+P 8075 3025
+F 0 "S1" H 8075 2850 60  0000 C CNN
+F 1 "EVQ-Q2S03W" H 8075 3250 60  0000 C CNN
+	1    8075 3025
+	1    0    0    -1
+$EndComp
 Text Label 3600 3950 0    40   ~ 0
 SPI_IRQ_RF

Commit message: Added foottprints for switches.
Parts:
- removed R25: 10k, symbol RES
- removed S5: EVQ-Q2S03W, symbol EVQ-Q2S03W
- R21, R22, R23, R24: value 10k -> 2.8k(1%)
Connections:
- net labels added: S1, S2, S3, S4
- wire segments 187 -> 204

Commit message: Merged dev_alex
Connections:
- net labels added: SPI1_IRQ_RF
Changed lines of the file:
@@
-EESchema Schematic File Version 2  date 9/7/2012 4:03:21 PM
+EESchema Schematic File Version 2  date Fri 07 Sep 2012 05:49:39 PM EDT
 LIBS:power
 LIBS:device
@@
 $EndComp
 Text Label 3600 3950 0    40   ~ 0
-SPI_IRQ_RF
-Text Label 4850 4250 2    40   ~ 0
+SPI1_IRQ_RF
+Text Label 7200 4050 0    40   ~ 0
 DEN_G
 Text Label 8000 1600 0    40   ~ 0
@@
 SPI1_MISO
 Text Label 9350 1250 2    60   ~ 0
-SPI_IRQ_RF
+SPI1_IRQ_RF
 Text Label 9350 1150 2    60   ~ 0
 SPI1_nCS_RF

Commit message: Rewired buttons
Parts:
- removed R21, R22, R23, R24: 2.8k(1%), symbol RES
Connections:
- wire segments 204 -> 199
Changed lines of the file:
@@
-EESchema Schematic File Version 2  date Fri 07 Sep 2012 05:49:39 PM EDT
+EESchema Schematic File Version 2  date Fri 07 Sep 2012 06:23:43 PM EDT
 LIBS:power
 LIBS:device
@@
 $EndDescr
 Wire Wire Line
-	8700 4625 8700 2925
-Wire Wire Line
 	5100 5350 4850 5350
 Wire Wire Line
@@
 Wire Wire Line
 	5100 4250 4850 4250
-Connection ~ 8700 3525
-Wire Wire Line
-	8550 3525 8700 3525
-Connection ~ 8700 4625
-Wire Wire Line
-	8700 4625 8550 4625
 Wire Wire Line
 	8400 3725 8250 3725
@@
 Wire Wire Line
 	8250 4825 8400 4825
-Wire Wire Line
-	8700 2925 8550 2925
-Connection ~ 8700 4075
-Wire Wire Line
-	8550 4075 8875 4075
 Wire Wire Line
 	7900 2925 7800 2925
@@
 Text Label 7800 2925 2    60   ~ 0
 S1
-Text GLabel 8875 4075 2    60   Input ~ 0
-Vreg
-$Comp
-L RES R24
-U 1 1 504A3CA3
-P 8400 4625
-F 0 "R24" H 8470 4590 50  0000 L TNN
-F 1 "2.8k(1%)" H 8500 4700 30  0000 C BNN
-	1    8400 4625
-	1    0    0    -1
-$EndComp
-$Comp
-L RES R23
-U 1 1 504A3CA0
-P 8400 4075
-F 0 "R23" H 8470 4040 50  0000 L TNN
-F 1 "2.8k(1%)" H 8500 4150 30  0000 C BNN
-	1    8400 4075
-	1    0    0    -1
-$EndComp
-$Comp
-L RES R22
-U 1 1 504A3C9C
-P 8400 3525
-F 0 "R22" H 8470 3490 50  0000 L TNN
-F 1 "2.8k(1%)" H 8500 3600 30  0000 C BNN
-	1    8400 3525
-	1    0    0    -1
-$EndComp
-$Comp
-L RES R21
-U 1 1 504A3C92
-P 8400 2925
-AR Path="/500B6AFA/504A3C92" Ref="R21"  Part="1"
-AR Path="/500B69F1/504A3C92" Ref="R21"  Part="1"
-F 0 "R21" H 8470 2890 50  0000 L TNN
-F 1 "2.8k(1%)" H 8400 2980 30  0000 C BNN
-	1    8400 2925
-	1    0    0    -1
-$EndComp
 $Comp
 L GND #PWR?

Commit message: Added step-up converter in the schematics files
Connections:
- net labels added: POW_NXT
- wire segments 199 -> 201

Commit message: Moved the hierarchical pins for the audio to a more appropriate place.
Parts:
- added J?: NXT_RJ12, symbol NXT_RJ12
Connections:
- net labels added: NXT_SCL, NXT_SDA, POW_9V, Vnxt4.3v
- wire segments 201 -> 241

Commit message: Added the switching mechanism fro the 9v line
Parts:
- added D?: DIODESCH, symbol DIODESCH
- added Q?: MOS_N, symbol MOS_N
- added R?: 100k, symbol RES
- added R?: 5k, symbol RES
- added R?: 12k, symbol RES
Connections:
- net labels added: Analog_POW, STM32_ADC, Vnxt9v
- wire segments 241 -> 227

Commit message: Assigned lots of footprints, added diode footprint
Parts:
- D1: renamed from D?; value DIODESCH -> RB520S30CT-ND
- Q1: renamed from Q?; value MOS_N -> 2N7002P
- gave numbers to parts that had none: 4
Changed lines of the file:
@@
-EESchema Schematic File Version 2  date 9/11/2012 11:18:24 AM
+EESchema Schematic File Version 2  date Wed 26 Sep 2012 06:41:48 PM EDT
 LIBS:power
 LIBS:device
@@
 Sheet 3 6
 Title ""
-Date "10 sep 2012"
+Date "26 sep 2012"
 Rev ""
 Comp ""
@@
 POW_9V
 $Comp
-L GND #PWR?
+L GND #PWR015
 U 1 1 504E596F
 P 9750 4450
-F 0 "#PWR?" H 9750 4450 30  0001 C CNN
+F 0 "#PWR015" H 9750 4450 30  0001 C CNN
 F 1 "GND" H 9750 4380 30  0001 C CNN
 	1    9750 4450
@@
 Analog_POW
 $Comp
-L RES R?
+L RES R7
 U 1 1 504E58A7
 P 9750 3500
-F 0 "R?" H 9820 3465 50  0000 L TNN
+F 0 "R7" H 9820 3465 50  0000 L TNN
 F 1 "12k" H 9750 3555 30  0000 C BNN
 	1    9750 3500
@@
 Vreg
 $Comp
-L DIODESCH D?
+L DIODESCH D1
 U 1 1 504E5806
 P 10500 4000
-F 0 "D?" H 10500 4100 40  0000 C CNN
-F 1 "DIODESCH" H 10500 3900 40  0000 C CNN
+F 0 "D1" H 10500 4100 40  0000 C CNN
+F 1 "RB520S30CT-ND" H 10500 3900 40  0000 C CNN
 	1    10500 4000
 	0    1    1    0
 $EndComp
 $Comp
-L RES R?
+L RES R8
 U 1 1 504E57D1
 P 10100 4050
-F 0 "R?" H 10170 4015 50  0000 L TNN
+F 0 "R8" H 10170 4015 50  0000 L TNN
 F 1 "5k" H 10050 4100 30  0000 C BNN
 	1    10100 4050
@@
 $EndComp
 $Comp
-L RES R?
+L RES R6
 U 1 1 504E57B0
 P 9250 4150
-F 0 "R?" H 9320 4115 50  0000 L TNN
+F 0 "R6" H 9320 4115 50  0000 L TNN
 F 1 "100k" H 9250 4205 30  0000 C BNN
 	1    9250 4150
@@
 $EndComp
 $Comp
-L MOS_N Q?
+L MOS_N Q1
 U 1 1 504E571E
 P 9650 3950
-F 0 "Q?" H 9660 4120 60  0000 R CNN
-F 1 "MOS_N" H 9660 3800 60  0000 R CNN
+F 0 "Q1" H 9660 4120 60  0000 R CNN
+F 1 "2N7002P" H 9660 3800 60  0000 R CNN
 	1    9650 3950
 	1    0    0    -1
@@
 Vnxt4.3v
 $Comp
-L GND #PWR?
+L GND #PWR016
 U 1 1 504E3C51
 P 9800 5500
-F 0 "#PWR?" H 9800 5500 30  0001 C CNN
+F 0 "#PWR016" H 9800 5500 30  0001 C CNN
 F 1 "GND" H 9800 5430 30  0001 C CNN
 	1    9800 5500
@@
 $EndComp
 $Comp
-L NXT_RJ12 J?
+L NXT_RJ12 J3
 U 1 1 504E3BFA
 P 9850 6100
-F 0 "J?" H 10050 6600 60  0000 C CNN
+F 0 "J3" H 10050 6600 60  0000 C CNN
 F 1 "NXT_RJ12" H 9700 6600 60  0000 C CNN
 	1    9850 6100
@@
 S1
 $Comp
-L GND #PWR?
+L GND #PWR017
 U 1 1 504A3C49
 P 8400 4825
-F 0 "#PWR?" H 8400 4825 30  0001 C CNN
+F 0 "#PWR017" H 8400 4825 30  0001 C CNN
 F 1 "GND" H 8400 4755 30  0001 C CNN
 	1    8400 4825
@@
 $EndComp
 $Comp
-L GND #PWR?
+L GND #PWR018
 U 1 1 504A3C3E
 P 8400 3725
-F 0 "#PWR?" H 8400 3725 30  0001 C CNN
+F 0 "#PWR018" H 8400 3725 30  0001 C CNN
 F 1 "GND" H 8400 3655 30  0001 C CNN
 	1    8400 3725
@@
 $EndComp
 $Comp
-L GND #PWR?
+L GND #PWR019
 U 1 1 504A3BFE
 P 8400 4275
-F 0 "#PWR?" H 8400 4275 30  0001 C CNN
+F 0 "#PWR019" H 8400 4275 30  0001 C CNN
 F 1 "GND" H 8400 4205 30  0001 C CNN
 	1    8400 4275
@@
 $EndComp
 $Comp
-L GND #PWR?
+L GND #PWR020
 U 1 1 504A3BF9
 P 8400 3125
-F 0 "#PWR?" H 8400 3125 30  0001 C CNN
+F 0 "#PWR020" H 8400 3125 30  0001 C CNN
 F 1 "GND" H 8400 3055 30  0001 C CNN
 	1    8400 3125
@@
 LCD_D0
 $Comp
-L GND #PWR015
+L GND #PWR021
 U 1 1 501885AA
 P 8050 1800
-F 0 "#PWR015" H 8050 1800 30  0001 C CNN
+F 0 "#PWR021" H 8050 1800 30  0001 C CNN
 F 1 "GND" H 8050 1730 30  0001 C CNN
 	1    8050 1800
@@
 Vreg
 $Comp
-L GND #PWR016
+L GND #PWR022
 U 1 1 50188517
 P 6150 1750
-F 0 "#PWR016" H 6150 1750 30  0001 C CNN
+F 0 "#PWR022" H 6150 1750 30  0001 C CNN
 F 1 "GND" H 6150 1680 30  0001 C CNN
 	1    6150 1750
@@
 $EndComp
 $Comp
-L GND #PWR017
+L GND #PWR023
 U 1 1 5010608D
 P 1750 2350
-F 0 "#PWR017" H 1750 2350 30  0001 C CNN
+F 0 "#PWR023" H 1750 2350 30  0001 C CNN
 F 1 "GND" H 1750 2280 30  0001 C CNN
 	1    1750 2350
@@
 $EndComp
 $Comp
-L GND #PWR018
+L GND #PWR024
 U 1 1 500D75A4
 P 2400 5900
-F 0 "#PWR018" H 2400 5900 30  0001 C CNN
+F 0 "#PWR024" H 2400 5900 30  0001 C CNN
 F 1 "GND" H 2400 5830 30  0001 C CNN
 	1    2400 5900
@@
 $EndComp
 $Comp
-L GND #PWR019
+L GND #PWR025
 U 1 1 500D7599
 P 6050 6000
-F 0 "#PWR019" H 6050 6000 30  0001 C CNN
+F 0 "#PWR025" H 6050 6000 30  0001 C CNN
 F 1 "GND" H 6050 5930 30  0001 C CNN
 	1    6050 6000
