File: pcb/discovery.sch (KiCad schematic (older format))
At the start: 6 parts, among them U1 FT230X, U2 STM32F4-DISCOVERY

Commit message: finished CPLD schematic and started adding new discovery sheet
Parts:
- removed U?: XC2C64A-XQFG48, symbol XC2C64A-XQFG48
- added S? (x4): EVQ-Q2S03W, symbol EVQ-Q2S03W
Connections:
- wire segments 187 -> 205
Other:
- note added: "CS43L22 RESET"
Changed lines of the file:
@@
-EESchema Schematic File Version 2  date Thu 06 Dec 2012 06:44:11 PM EST
+EESchema Schematic File Version 2  date 12/12/2012 5:26:02 PM
 LIBS:power
 LIBS:device
@@
 $Descr A4 11700 8267
 encoding utf-8
-Sheet 2 8
+Sheet 3 10
 Title ""
-Date "6 dec 2012"
+Date "12 dec 2012"
 Rev ""
 Comp ""
@@
 Comment4 ""
 $EndDescr
-Wire Wire Line
-	5850 7600 5850 7500
+$Sheet
+S -4250 4450 1800 5750
+U 50C90435
+F0 "disc" 60
+F1 "disc.sch" 60
+$EndSheet
+Text Notes 9000 2800 0    50   ~ 0
+CS43L22 RESET
+Wire Wire Line
+	8850 5975 8750 5975
+Wire Wire Line
+	9200 6175 9200 6300
+Wire Wire Line
+	8850 5625 8850 5750
+Wire Wire Line
+	8850 5750 9200 5750
+Wire Wire Line
+	9200 5750 9200 5625
+Wire Wire Line
+	8850 4825 8750 4825
+Wire Wire Line
+	9350 6725 9200 6725
+Wire Wire Line
+	9200 6175 9350 6175
+Wire Wire Line
+	9350 5025 9200 5025
+Wire Wire Line
+	9200 5625 9350 5625
+Wire Wire Line
+	9200 5025 9200 5150
+Wire Wire Line
+	9200 5150 8850 5150
+Wire Wire Line
+	8850 5150 8850 5025
+Wire Wire Line
+	9200 6300 8850 6300
+Wire Wire Line
+	8850 6300 8850 6175
+Wire Wire Line
+	9200 6725 9200 6850
+Wire Wire Line
+	9200 6850 8850 6850
+Wire Wire Line
+	8850 6850 8850 6725
+Wire Wire Line
+	8850 6525 8750 6525
+Wire Wire Line
+	8725 5425 8850 5425
+$Comp
+L EVQ-Q2S03W S?
+U 1 1 50C8E84F
+P 9025 4925
+F 0 "S?" H 9025 4750 60  0000 C CNN
+F 1 "EVQ-Q2S03W" H 9025 5150 60  0000 C CNN
+	1    9025 4925
+	1    0    0    -1
+$EndComp
+$Comp
+L EVQ-Q2S03W S?
+U 1 1 50C8E84E
+P 9025 5525
+F 0 "S?" H 9025 5350 60  0000 C CNN
+F 1 "EVQ-Q2S03W" H 9025 5725 60  0000 C CNN
+	1    9025 5525
+	1    0    0    -1
+$EndComp
+$Comp
+L EVQ-Q2S03W S?
+U 1 1 50C8E84D
+P 9025 6075
+F 0 "S?" H 9025 5900 60  0000 C CNN
+F 1 "EVQ-Q2S03W" H 9025 6275 60  0000 C CNN
+	1    9025 6075
+	1    0    0    -1
+$EndComp
+$Comp
+L EVQ-Q2S03W S?
+U 1 1 50C8E84C
+P 9025 6625
+F 0 "S?" H 9025 6450 60  0000 C CNN
+F 1 "EVQ-Q2S03W" H 9025 6850 60  0000 C CNN
+	1    9025 6625
+	1    0    0    -1
+$EndComp
+$Comp
+L GND #PWR?
+U 1 1 50C8E84B
+P 9350 5025
+F 0 "#PWR?" H 9350 5025 30  0001 C CNN
+F 1 "GND" H 9350 4955 30  0001 C CNN
+	1    9350 5025
+	0    -1   1    0
+$EndComp
+$Comp
+L GND #PWR?
+U 1 1 50C8E84A
+P 9350 6175
+F 0 "#PWR?" H 9350 6175 30  0001 C CNN
+F 1 "GND" H 9350 6105 30  0001 C CNN
+	1    9350 6175
+	0    -1   1    0
+$EndComp
+$Comp
+L GND #PWR?
+U 1 1 50C8E849
+P 9350 5625
+F 0 "#PWR?" H 9350 5625 30  0001 C CNN
+F 1 "GND" H 9350 5555 30  0001 C CNN
+	1    9350 5625
+	0    -1   1    0
+$EndComp
+$Comp
+L GND #PWR?
+U 1 1 50C8E848
+P 9350 6725
+F 0 "#PWR?" H 9350 6725 30  0001 C CNN
+F 1 "GND" H 9350 6655 30  0001 C CNN
+	1    9350 6725
+	0    -1   1    0
+$EndComp
+Text Label 8750 4825 2    60   ~ 0
+S1
+Text Label 8725 5425 2    60   ~ 0
+S2
+Text Label 8750 5975 2    60   ~ 0
+S3
+Text Label 8750 6525 2    60   ~ 0
+S4
 Wire Wire Line
 	6950 3500 7050 3500
@@
 Wire Wire Line
 	9050 3500 8950 3500
-Wire Wire Line
-	5850 5150 5850 5200
-Text GLabel 5850 7600 3    60   Input ~ 0
-Vreg
-Text GLabel 5850 5150 1    60   Input ~ 0
-Vreg
 Text HLabel 6950 3500 0    60   Output ~ 0
 NXT_SCL
@@
 	1    0    0    -1
 $EndComp
-$Comp
-L XC2C64A-XQFG48 U?
-U 1 1 50C11989
-P 5800 6350
-F 0 "U?" H 6500 5200 60  0000 C CNN
-F 1 "XC2C64A-XQFG48" H 6850 7500 60  0000 C CNN
-	1    5800 6350
-	1    0    0    -1
-$EndComp

Commit message: Removed the POW multiplexer lines and put the standard interrupt lines
Connections:
- net labels added: EXTI0, EXTI1, EXTI2, EXTI3, EXTI4, EXTI5, EXTI6, EXTI7, EXTI8, EXTI9
- net labels removed: SPI_IRQ_RF, SPI_IRQ_TOUCH
- wire segments 205 -> 201
Other:
- note added: "CS43L22"
- note removed: "CS43L22 RESET"

Commit message: Rearranged all the lines except for the power lines.
Connections:
- net labels added: NXT_ADC, SPI_nCS_ACC, SPI_nCS_CPLD, SPI_nCS_GYR
- net labels removed: DRDYg/INT2_G, INT1_A, INT1_G, INT2_A, STM32_ADC
- wire segments 201 -> 206
Other:
- note added: "Audio"
- note added: "External Interrupts"
- note added: "LCD I/O"
- note added: "NXT I/O"
- note added: "Power Status and Enable"
- note added: "Suggested Interrupt Setup:\nIndependent Vectors:\n EXTI0: LIS302_INT1\n EXTI1: LIS302_INT2\n EXTI2: SPI_IRQ_RF\n EXTI3: SPI_IRQ_TOUCH\n EXTI4:\n\nEXTI9_5:\n EXTI5: S1\n EXTI6: S2\n EXTI7: S3\n EXTI8: S4\n EXTI9:\n\nEXTI15_10:\n EXTI10: \n EXTI11: INT1_A\n EXTI12: INT1_G\n EXTI13: INT2_A\n EXTI14: \n EXTI15: DRDYg/INT2_G"
- note removed: "Interrupts:\nIndependent Vectors:\n EXTI0: LIS302_INT1\n EXTI1: LIS302_INT2\n EXTI2: SPI_IRQ_RF\n EXTI3: SPI_IRQ_TOUCH\n EXTI4:\n\nEXTI9_5:\n EXTI5: S1\n EXTI6: S2\n EXTI7: S3\n EXTI8: S4\n EXTI9:\n\nEXTI15_10:\n EXTI10: \n EXTI11: INT1_A\n EXTI12: INT1_G\n EXTI13: INT2_A\n EXTI14: \n EXTI15: DRDYg/INT2_G"

Commit message: CPLD connection finished.
Connections:
- net labels added: EXTI11, EXTI12, EXTI13, EXTI15
- net labels removed: EN_POW_NXT, EXTI9, POW_HPWR, POW_MODE
- wire segments 206 -> 207
- no-connect marks 22 -> 27
Other:
- note added: "SWO"

Commit message: Switched the interrupt line location so that we can use one of the ADC channels for the audio.
Parts:
- removed S? (x4): EVQ-Q2S03W, symbol EVQ-Q2S03W
Connections:
- net labels removed: S1, S2, S3, S4
- wire segments 207 -> 187
Other:
- note added: "ADC12_IN15"
Changed lines of the file:
@@
-EESchema Schematic File Version 2  date 12/19/2012 4:02:29 PM
+EESchema Schematic File Version 2  date 12/19/2012 4:17:57 PM
 LIBS:power
 LIBS:device
@@
 Comment4 ""
 $EndDescr
+Text Notes 2450 2000 0    40   ~ 0
+ADC12_IN15
 Text Notes 9000 2600 0    50   ~ 0
 SWO
@@
 Wire Wire Line
 	6950 3500 7050 3500
-Wire Wire Line
-	10025 5425 10150 5425
-Wire Wire Line
-	10150 6525 10050 6525
-Wire Wire Line
-	10150 6725 10150 6850
-Wire Wire Line
-	10150 6850 10500 6850
-Wire Wire Line
-	10500 6850 10500 6725
-Wire Wire Line
-	10150 6175 10150 6300
-Wire Wire Line
-	10150 6300 10500 6300
-Wire Wire Line
-	10150 5025 10150 5150
-Wire Wire Line
-	10150 5150 10500 5150
-Wire Wire Line
-	10500 5150 10500 5025
-Wire Wire Line
-	10650 5625 10500 5625
-Wire Wire Line
-	10500 5025 10650 5025
-Wire Wire Line
-	10650 6175 10500 6175
-Wire Wire Line
-	10500 6725 10650 6725
-Wire Wire Line
-	10150 4825 10050 4825
-Wire Wire Line
-	10500 5625 10500 5750
-Wire Wire Line
-	10500 5750 10150 5750
-Wire Wire Line
-	10150 5750 10150 5625
-Wire Wire Line
-	10500 6175 10500 6300
-Wire Wire Line
-	10150 5975 10050 5975
 Wire Wire Line
 	4050 6150 4200 6150
@@
 Text Notes 9000 2800 0    50   ~ 0
 CS43L22
-$Comp
-L EVQ-Q2S03W S?
-U 1 1 50C8E84F
-P 10325 4925
-F 0 "S?" H 10325 4750 60  0000 C CNN
-F 1 "EVQ-Q2S03W" H 10325 5150 60  0000 C CNN
-	1    10325 4925
-	1    0    0    -1
-$EndComp
-$Comp
-L EVQ-Q2S03W S?
-U 1 1 50C8E84E
-P 10325 5525
-F 0 "S?" H 10325 5350 60  0000 C CNN
-F 1 "EVQ-Q2S03W" H 10325 5725 60  0000 C CNN
-	1    10325 5525
-	1    0    0    -1
-$EndComp
-$Comp
-L EVQ-Q2S03W S?
-U 1 1 50C8E84D
-P 10325 6075
-F 0 "S?" H 10325 5900 60  0000 C CNN
-F 1 "EVQ-Q2S03W" H 10325 6275 60  0000 C CNN
-	1    10325 6075
-	1    0    0    -1
-$EndComp
-$Comp
-L EVQ-Q2S03W S?
-U 1 1 50C8E84C
-P 10325 6625
-F 0 "S?" H 10325 6450 60  0000 C CNN
-F 1 "EVQ-Q2S03W" H 10325 6850 60  0000 C CNN
-	1    10325 6625
-	1    0    0    -1
-$EndComp
-$Comp
-L GND #PWR?
-U 1 1 50C8E84B
-P 10650 5025
-F 0 "#PWR?" H 10650 5025 30  0001 C CNN
-F 1 "GND" H 10650 4955 30  0001 C CNN
-	1    10650 5025
-	0    -1   1    0
-$EndComp
-$Comp
-L GND #PWR?
-U 1 1 50C8E84A
-P 10650 6175
-F 0 "#PWR?" H 10650 6175 30  0001 C CNN
-F 1 "GND" H 10650 6105 30  0001 C CNN
-	1    10650 6175
-	0    -1   1    0
-$EndComp
-$Comp
-L GND #PWR?
-U 1 1 50C8E849
-P 10650 5625
-F 0 "#PWR?" H 10650 5625 30  0001 C CNN
-F 1 "GND" H 10650 5555 30  0001 C CNN
-	1    10650 5625
-	0    -1   1    0
-$EndComp
-$Comp
-L GND #PWR?
-U 1 1 50C8E848
-P 10650 6725
-F 0 "#PWR?" H 10650 6725 30  0001 C CNN
-F 1 "GND" H 10650 6655 30  0001 C CNN
-	1    10650 6725
-	0    -1   1    0
-$EndComp
-Text Label 10050 4825 2    60   ~ 0
-S1
-Text Label 10025 5425 2    60   ~ 0
-S2
-Text Label 10050 5975 2    60   ~ 0
-S3
-Text Label 10050 6525 2    60   ~ 0
-S4
 Text HLabel 6950 3500 0    60   Output ~ 0
 NXT_SCL
@@
 Text Label 3150 1500 2    40   ~ 0
 STM32_ADC_CH11
+Text Label 6800 2300 2    40   ~ 0
+EN_POW_9V
 Text Label 9150 2000 0    40   ~ 0
-EN_POW_9V
-Text Label 3150 2000 2    40   ~ 0
 EXTI5
 Text Label 6800 3700 2    40   ~ 0
@@
 Text Label 2550 6150 2    60   ~ 0
 AUDIO_IN_R
-Text Label 2550 6050 2    60   ~ 0
+Text Label 3150 2000 2    40   ~ 0
 AUDIO_IN_L
 Text HLabel 7900 6200 2    60   BiDi ~ 0

Commit message: Added backlight driver, connected to I2C1, annotated stuff
Connections:
- net labels added: BKLT_EN, I2C1_SDA
- wire segments 187 -> 190
Other:
- note added: "I2C1"

Commit message: Modified labels on discover.sch and rearranged sheet disposition in the top-level schematic.
Connections:
- net labels added: I2C3_SCL, I2C3_SDA, STM32_ADC_CH15
- net labels removed: NXT_SCL, NXT_SDA
Other:
- note removed: "ADC12_IN15"
Changed lines of the file:
@@
-EESchema Schematic File Version 2  date Fri 28 Dec 2012 12:18:10 AM EST
+EESchema Schematic File Version 2  date 12/30/2012 6:01:05 PM
 LIBS:power
 LIBS:device
@@
 $Descr A4 11700 8267
 encoding utf-8
-Sheet 2 9
+Sheet 3 9
 Title ""
-Date "28 dec 2012"
+Date "30 dec 2012"
 Rev ""
 Comp ""
@@
 $EndDescr
 Wire Notes Line
+	1750 6200 3300 6200
+Wire Wire Line
+	6200 6150 5600 6150
+Wire Notes Line
 	8850 6200 8850 5900
 Wire Notes Line
@@
 	9300 6100 9450 6100
 Wire Wire Line
-	1450 7150 1300 7150
-Wire Wire Line
-	1450 7350 1300 7350
-Wire Wire Line
-	1450 7250 1300 7250
+	1050 7150 900  7150
+Wire Wire Line
+	1050 7350 900  7350
+Wire Wire Line
+	1050 7250 900  7250
 Wire Wire Line
 	9150 2900 8950 2900
@@
 	5400 3000 5550 3000
 Wire Notes Line
-	1800 5900 1000 5900
-Wire Notes Line
-	2000 6200 2000 5900
-Wire Notes Line
-	2000 6200 3300 6200
+	1400 5900 600  5900
+Wire Notes Line
+	1750 6200 1750 5900
 Wire Notes Line
 	3300 6200 3300 5900
 Wire Notes Line
-	3300 5900 2000 5900
-Wire Notes Line
 	7000 6900 7000 5900
 Wire Notes Line
@@
 	8700 5900 7000 5900
 Wire Wire Line
-	1450 6850 1300 6850
-Wire Wire Line
-	1300 6550 1450 6550
-Wire Wire Line
-	1450 6650 1300 6650
-Wire Wire Line
-	1300 6750 1450 6750
-Wire Wire Line
-	1300 6450 1450 6450
-Wire Wire Line
-	1300 6050 1450 6050
+	1050 6850 900  6850
+Wire Wire Line
+	900  6550 1050 6550
+Wire Wire Line
+	1050 6650 900  6650
+Wire Wire Line
+	900  6750 1050 6750
+Wire Wire Line
+	900  6450 1050 6450
+Wire Wire Line
+	900  6050 1050 6050
 Wire Wire Line
 	5300 7050 5500 7050
@@
 	7900 6500 7750 6500
 Wire Wire Line
-	1300 6350 1450 6350
-Wire Wire Line
-	6200 6150 5950 6150
+	900  6350 1050 6350
 Wire Wire Line
 	4100 7000 4250 7000
@@
 	2700 6050 2550 6050
 Wire Wire Line
-	1450 6250 1300 6250
+	1050 6250 900  6250
 Wire Wire Line
 	2750 7000 2900 7000
@@
 	6200 6250 5950 6250
 Wire Wire Line
-	6200 6050 5950 6050
-Wire Wire Line
 	7900 6000 7750 6000
 Wire Wire Line
@@
 	4050 6150 4200 6150
 Wire Wire Line
-	1300 6150 1450 6150
+	900  6150 1050 6150
 Wire Wire Line
 	5400 2300 5550 2300
@@
 	3300 2700 3150 2700
 Wire Wire Line
-	1450 7050 1300 7050
+	1050 7050 900  7050
 Wire Wire Line
 	7900 6800 7750 6800
 Wire Wire Line
 	9450 6000 9300 6000
+Wire Wire Line
+	6200 6050 5600 6050
+Wire Notes Line
+	3300 5900 1750 5900
+Text Label 2550 6050 2    60   ~ 0
+STM32_ADC_CH15
+Text Label 9050 3500 0    40   ~ 0
+I2C3_SDA
+Text Label 6950 3500 2    40   ~ 0
+I2C3_SCL
+Text HLabel 6200 6050 2    60   BiDi ~ 0
+I2C3_SDA
+Text HLabel 6200 6150 2    60   BiDi ~ 0
+I2C3_SCL
+Text Label 5600 6050 2    60   ~ 0
+I2C3_SDA
+Text Label 5600 6150 2    60   ~ 0
+I2C3_SCL
 Text Label 9300 6100 2    60   ~ 0
 I2C1_SCL
@@
 Text HLabel 9450 6000 2    60   BiDi ~ 0
 I2C1_SDA
-Text Notes 2450 2000 0    40   ~ 0
-ADC12_IN15
 Text Notes 9000 2600 0    50   ~ 0
 SWO
-Text Label 1300 7150 2    60   ~ 0
+Text Label 900  7150 2    60   ~ 0
 EXTI12
-Text HLabel 1450 7150 2    60   Input ~ 0
+Text HLabel 1050 7150 2    60   Input ~ 0
 EXTI12
 Text Label 5550 3000 0    40   ~ 0
@@
 NoConn ~ 5400 1500
 NoConn ~ 7050 2400
-Text Label 1300 7350 2    60   ~ 0
+Text Label 900  7350 2    60   ~ 0
 EXTI15
-Text HLabel 1450 7350 2    60   Input ~ 0
+Text HLabel 1050 7350 2    60   Input ~ 0
 EXTI15
 Text Label 9150 3200 0    40   ~ 0
 EXTI15
-Text HLabel 1450 7250 2    60   Input ~ 0
+Text HLabel 1050 7250 2    60   Input ~ 0
 EXTI13
-Text Label 1300 7250 2    60   ~ 0
+Text Label 900  7250 2    60   ~ 0
 EXTI13
 Text Label 9150 1900 0    40   ~ 0
 EXTI13
-Text HLabel 1450 7050 2    60   Input ~ 0
+Text HLabel 1050 7050 2    60   Input ~ 0
 EXTI11
-Text Label 1300 7050 2    60   ~ 0
+Text Label 900  7050 2    60   ~ 0
 EXTI11
 Text Label 9150 3100 0    40   ~ 0
@@
 Text Label 2750 7300 2    60   ~ 0
 SPI_nCS_GYR
-Text Notes 1000 5900 0    60   ~ 0
+Text Notes 600  5900 0    60   ~ 0
 External Interrupts
 Text Notes 3500 5900 0    60   ~ 0
@@
 Text Label 6800 2600 2    40   ~ 0
 DEN_G
-Text HLabel 1450 6850 2    60   Input ~ 0
+Text HLabel 1050 6850 2    60   Input ~ 0
 EXTI8
-Text Label 1300 6850 2    60   ~ 0
+Text Label 900  6850 2    60   ~ 0
 EXTI8
-Text Label 1300 6650 2    60   ~ 0
+Text Label 900  6650 2    60   ~ 0
 EXTI6
-Text HLabel 1450 6650 2    60   Input ~ 0
+Text HLabel 1050 6650 2    60   Input ~ 0
 EXTI6
-Text Label 1300 6750 2    60   ~ 0
+Text Label 900  6750 2    60   ~ 0
 EXTI7
-Text HLabel 1450 6750 2    60   Input ~ 0
+Text HLabel 1050 6750 2    60   Input ~ 0
 EXTI7
-Text Label 1300 6550 2    60   ~ 0
+Text Label 900  6550 2    60   ~ 0
 EXTI5
-Text HLabel 1450 6550 2    60   Input ~ 0
+Text HLabel 1050 6550 2    60   Input ~ 0
 EXTI5
-Text HLabel 1450 6450 2    60   Input ~ 0
+Text HLabel 1050 6450 2    60   Input ~ 0
 EXTI4
-Text Label 1300 6450 2    60   ~ 0
+Text Label 900  6450 2    60   ~ 0
 EXTI4
-Text Label 1300 6050 2    60   ~ 0
+Text Label 900  6050 2    60   ~ 0
 EXTI0
-Text HLabel 1450 6050 2    60   Input ~ 0
+Text HLabel 1050 6050 2    60   Input ~ 0
 EXTI0
-Text HLabel 1450 6150 2    60   Input ~ 0
+Text HLabel 1050 6150 2    60   Input ~ 0
 EXTI1
 Text HLabel 5500 7050 2    60   Output ~ 0
@@
 Text Label 6800 2000 2    40   ~ 0
 EXTI4
-Text Label 1300 6150 2    60   ~ 0
+Text Label 900  6150 2    60   ~ 0
 EXTI1
 Text Label 3150 2100 2    40   ~ 0
@@
 Text Notes 9000 2800 0    50   ~ 0
 CS43L22
-Text HLabel 6950 3500 0    60   Output ~ 0
-NXT_SCL
-Text HLabel 9050 3500 2    60   Output ~ 0
-NXT_SDA
 Text HLabel 5550 3100 2    60   Input ~ 0
 SPI2_MISO
@@
 Text HLabel 7900 6300 2    60   Output ~ 0
 LCD_nRS
-Text HLabel 1450 6350 2    60   Input ~ 0
+Text HLabel 1050 6350 2    60   Input ~ 0
 EXTI3
 Text HLabel 7900 6000 2    60   Output ~ 0
 SPI_nCS_TOUCH
-Text Label 1300 6350 2    60   ~ 0
+Text Label 900  6350 2    60   ~ 0
 EXTI3
 Text Label 7750 6000 2    60   ~ 0
@@
 Text HLabel 6200 6250 2    60   Input ~ 0
 NXT_ADC
-Text HLabel 6200 6150 2    60   BiDi ~ 0
-NXT_SCL
-Text HLabel 6200 6050 2    60   BiDi ~ 0
-NXT_SDA
 Text Label 5950 6250 2    60   ~ 0
 STM32_ADC_CH11
-Text Label 5950 6150 2    60   ~ 0
-NXT_SCL
-Text Label 5950 6050 2    60   ~ 0
-NXT_SDA
 Text Label 4050 6300 2    60   ~ 0
 EN_POW_9V
@@
 AUDIO_IN_R
 Text Label 3150 2000 2    40   ~ 0
-AUDIO_IN_L
+STM32_ADC_CH15
 Text HLabel 7900 6200 2    60   BiDi ~ 0
 LCD_D[0..15]
-Text HLabel 1450 6250 2    60   Input ~ 0
+Text HLabel 1050 6250 2    60   Input ~ 0
 EXTI2
 Text HLabel 2900 7100 2    60   Output ~ 0
@@
 Text HLabel 2900 7000 2    60   Output ~ 0
 RF_RESET
-Text Label 1300 6250 2    60   ~ 0
+Text Label 900  6250 2    60   ~ 0
 EXTI2
 Text Label 2750 7100 2    60   ~ 0
