File: pcb/power.sch (KiCad schematic (older format))
At the start: 21 parts, among them U2 LTC3559, U6 USBMICROCONN

Commit message: Added a pull-down for the enable as well as changed the supply to Vbat from Vreg
Parts:
- added R?: 10k, symbol RES
Connections:
- wire segments 100 -> 78
Other:
- moved on the sheet: C?, L2, R?
Changed lines of the file:
@@
-EESchema Schematic File Version 2  date 9/9/2012 8:55:02 PM
+EESchema Schematic File Version 2  date 9/10/2012 1:18:59 PM
 LIBS:power
 LIBS:device
@@
 LIBS:valves
 LIBS:f4_daughter
-LIBS:f4_daughter-cache
 EELAYER 25  0
 EELAYER END
@@
 Comment4 ""
 $EndDescr
-Wire Wire Line
-	8400 2900 8700 2900
-Wire Wire Line
-	8700 2600 7700 2600
-Connection ~ 10100 2600
-Wire Wire Line
-	9900 2900 10100 2900
-Wire Wire Line
-	10000 2300 10000 2100
-Wire Wire Line
-	10000 2300 9900 2300
+Connection ~ 8250 1900
+Wire Wire Line
+	8250 1950 8250 1900
+Wire Wire Line
+	8100 1900 8400 1900
+Wire Wire Line
+	8400 1600 7400 1600
+Connection ~ 9800 1600
+Wire Wire Line
+	9600 1900 9800 1900
+Wire Wire Line
+	9700 1300 9700 1100
+Wire Wire Line
+	9700 1300 9600 1300
 Connection ~ 5900 4100
 Wire Wire Line
-	6300 4100 5900 4100
-Wire Wire Line
-	5900 4100 5800 4100
-Wire Wire Line
-	5800 4100 5650 4100
+	6300 4100 5650 4100
 Wire Wire Line
 	6300 4100 6300 4000
@@
 Connection ~ 3800 2650
 Wire Wire Line
-	4900 2650 3800 2650
-Wire Wire Line
-	3800 2650 3650 2650
-Wire Wire Line
-	3800 2650 3800 2950
+	3650 2650 4900 2650
+Wire Wire Line
+	3800 2950 3800 2650
 Connection ~ 2700 2100
 Wire Wire Line
@@
 	3150 2400 3150 2500
 Wire Wire Line
-	3150 2500 2700 2500
-Wire Wire Line
-	2700 2500 2400 2500
+	3150 2500 2400 2500
 Wire Wire Line
 	3150 2200 3150 2100
@@
 	5900 1850 6100 1850
 Wire Wire Line
-	6100 1850 6100 2050
-Wire Wire Line
-	6100 2050 6100 2100
+	6100 1850 6100 2100
 Wire Wire Line
 	5600 1850 5450 1850
@@
 	5450 1850 5450 2100
 Wire Wire Line
-	4250 3800 4250 4100
-Wire Wire Line
-	4250 4100 4250 4150
+	4250 4150 4250 3800
 Wire Wire Line
 	4250 3100 4250 3050
 Wire Wire Line
-	4250 3050 4350 3050
-Wire Wire Line
-	4350 3050 4450 3050
-Wire Wire Line
-	4700 3350 4650 3350
-Wire Wire Line
-	4650 3350 4450 3350
+	4250 3050 4450 3050
+Wire Wire Line
+	4450 3350 4700 3350
 Wire Wire Line
 	5250 3100 5250 3150
@@
 	5350 3350 5350 3100
 Wire Wire Line
-	4250 3400 4250 3450
-Wire Wire Line
-	4250 3450 4250 3500
+	4250 3500 4250 3400
 Wire Wire Line
 	4250 3450 4050 3450
@@
 	4050 3450 4050 2750
 Wire Wire Line
-	4050 2750 4350 2750
-Wire Wire Line
-	4350 2750 4900 2750
+	4050 2750 4900 2750
 Wire Wire Line
 	5550 2100 5550 2050
@@
 	5250 1950 5250 2100
 Wire Wire Line
-	4450 3050 4450 3350
-Wire Wire Line
-	4450 3350 4450 3500
+	4450 3050 4450 3500
 Connection ~ 4450 3350
 Wire Wire Line
@@
 Connection ~ 4350 2750
 Wire Wire Line
-	4650 3150 4650 3350
-Wire Wire Line
-	4650 3350 4650 3500
-Wire Wire Line
-	5450 3100 5450 3300
-Wire Wire Line
-	5450 3300 5450 3400
+	4650 3500 4650 3150
+Wire Wire Line
+	5450 3400 5450 3100
 Wire Wire Line
 	2700 2650 2700 2500
 Wire Wire Line
-	3150 2100 2700 2100
-Wire Wire Line
-	2700 2100 2400 2100
+	3150 2100 2400 2100
 Wire Wire Line
 	3800 3250 3800 4100
 Wire Wire Line
-	3800 4100 4250 4100
-Wire Wire Line
-	4250 4100 4450 4100
-Wire Wire Line
-	4450 4100 4650 4100
+	3800 4100 4650 4100
 Wire Wire Line
 	5000 1750 5350 1750
@@
 	5900 2550 6050 2550
 Wire Wire Line
-	6050 2550 6050 2750
-Wire Wire Line
-	6050 2750 6050 2900
-Wire Wire Line
-	6050 2900 6050 2950
+	6050 2550 6050 2950
 Connection ~ 6050 2750
 Wire Wire Line
@@
 	6300 3400 6300 3300
 Wire Wire Line
-	6300 3300 5900 3300
-Wire Wire Line
-	5900 3300 5650 3300
-Wire Wire Line
-	5650 3300 5450 3300
+	6300 3300 5450 3300
 Connection ~ 5900 3300
 Wire Wire Line
-	8700 2300 8400 2300
-Wire Wire Line
-	7800 2300 7700 2300
-Wire Wire Line
-	7700 2300 7600 2300
-Wire Wire Line
-	7600 2300 7600 2100
-Wire Wire Line
-	7700 2300 7700 2400
-Connection ~ 7700 2300
-Connection ~ 7700 2600
-Wire Wire Line
-	10100 2900 10100 3000
-Wire Wire Line
-	10100 3450 10100 3300
-Wire Wire Line
-	10350 2600 10350 2650
-Wire Wire Line
-	10350 3000 10350 2850
-Wire Wire Line
-	10550 2600 10350 2600
-Wire Wire Line
-	10350 2600 10100 2600
-Wire Wire Line
-	10100 2600 9900 2600
-Connection ~ 10350 2600
-Wire Wire Line
-	7700 2600 7700 2800
-Wire Wire Line
-	10000 2100 7600 2100
-Wire Wire Line
-	7600 2100 7500 2100
-Connection ~ 7600 2100
-Text HLabel 8400 2900 0    60   Input ~ 0
+	8400 1300 8100 1300
+Wire Wire Line
+	7500 1300 7300 1300
+Wire Wire Line
+	7300 1300 7300 1100
+Wire Wire Line
+	7400 1400 7400 1300
+Connection ~ 7400 1300
+Connection ~ 7400 1600
+Wire Wire Line
+	9800 1900 9800 2000
+Wire Wire Line
+	9800 2450 9800 2300
+Wire Wire Line
+	10050 1600 10050 1650
+Wire Wire Line
+	10050 2000 10050 1850
+Wire Wire Line
+	9600 1600 10250 1600
+Connection ~ 10050 1600
+Wire Wire Line
+	7400 1600 7400 1800
+Wire Wire Line
+	9700 1100 7200 1100
+Connection ~ 7300 1100
+Wire Wire Line
+	8250 2250 8250 2400
+$Comp
+L GND #PWR?
+U 1 1 504E1CB3
+P 8250 2400
+F 0 "#PWR?" H 8250 2400 30  0001 C CNN
+F 1 "GND" H 8250 2330 30  0001 C CNN
+	1    8250 2400
+	1    0    0    -1
+$EndComp
+$Comp
+L RES R?
+U 1 1 504E1CAF
+P 8250 2100
+F 0 "R?" H 8320 2065 50  0000 L TNN
+F 1 "10k" H 8250 2155 30  0000 C BNN
+	1    8250 2100
+	0    -1   -1   0
+$EndComp
+Text HLabel 8100 1900 0    60   Input ~ 0
 POW_NXT
-Text GLabel 10550 2600 2    60   Output ~ 0
+Text GLabel 10250 1600 2    60   Output ~ 0
 Vnxt
-Text GLabel 7500 2100 0    60   Input ~ 0
-Vreg
+Text GLabel 7200 1100 0    60   Input ~ 0
+Vbat
 $Comp
 L GND #PWR?
 U 1 1 504D34F8
-P 10350 3000
-F 0 "#PWR?" H 10350 3000 30  0001 C CNN
-F 1 "GND" H 10350 2930 30  0001 C CNN
-	1    10350 3000
+P 10050 2000
+F 0 "#PWR?" H 10050 2000 30  0001 C CNN
+F 1 "GND" H 10050 1930 30  0001 C CNN
+	1    10050 2000
 	1    0    0    -1
 $EndComp
@@
 L CAP C?
 U 1 1 504D34CB
-P 10350 2750
-F 0 "C?" H 10370 2720 50  0000 L TNN
-F 1 "10u" H 10375 2770 30  0000 L BNN
-	1    10350 2750
+P 10050 1750
+F 0 "C?" H 10070 1720 50  0000 L TNN
+F 1 "10u" H 10075 1770 30  0000 L BNN
+	1    10050 1750
 	0    -1   -1   0
 $EndComp
@@
 L GND #PWR?
 U 1 1 504D341F
-P 10100 3450
-F 0 "#PWR?" H 10100 3450 30  0001 C CNN
-F 1 "GND" H 10100 3380 30  0001 C CNN
-	1    10100 3450
+P 9800 2450
+F 0 "#PWR?" H 9800 2450 30  0001 C CNN
+F 1 "GND" H 9800 2380 30  0001 C CNN
+	1    9800 2450
 	1    0    0    -1
 $EndComp
@@
 L RES R?
 U 1 1 504D340B
-P 10100 3150
-F 0 "R?" H 10170 3115 50  0000 L TNN
-F 1 "131k" H 10100 3205 30  0000 C BNN
-	1    10100 3150
+P 9800 2150
+F 0 "R?" H 9870 2115 50  0000 L TNN
+F 1 "131k" H 9800 2205 30  0000 C BNN
+	1    9800 2150
 	0    -1   -1   0
 $EndComp
@@
 L RES R?
 U 1 1 504D33DF
-P 10100 2750
-F 0 "R?" H 10170 2715 50  0000 L TNN
-F 1 "1M" H 10100 2805 30  0000 C BNN
-	1    10100 2750
+P 9800 1750
+F 0 "R?" H 9870 1715 50  0000 L TNN
+F 1 "1M" H 9800 1805 30  0000 C BNN
+	1    9800 1750
 	0    -1   -1   0
 $EndComp
@@
 L GND #PWR?
 U 1 1 504D3361
-P 7700 2800
-F 0 "#PWR?" H 7700 2800 30  0001 C CNN
-F 1 "GND" H 7700 2730 30  0001 C CNN
-	1    7700 2800
+P 7400 1800
+F 0 "#PWR?" H 7400 1800 30  0001 C CNN
+F 1 "GND" H 7400 1730 30  0001 C CNN
+	1    7400 1800
 	1    0    0    -1
 $EndComp
@@
 L CAP C?
 U 1 1 504D3316
-P 7700 2500
-F 0 "C?" H 7720 2470 50  0000 L TNN
-F 1 "10u" H 7725 2520 30  0000 L BNN
-	1    7700 2500
+P 7400 1500
+F 0 "C?" H 7420 1470 50  0000 L TNN
+F 1 "10u" H 7425 1520 30  0000 L BNN
+	1    7400 1500
 	0    1    1    0
 $EndComp
@@
 L INDUCTOR L2
 U 1 1 504D325B
-P 8100 2300
-F 0 "L2" V 8050 2300 40  0000 C CNN
-F 1 "CVH252009-4R7MCT-ND" V 8200 2300 30  0000 C CNN
-	1    8100 2300
+P 7800 1300
+F 0 "L2" V 7750 1300 40  0000 C CNN
+F 1 "CVH252009-4R7MCT-ND" V 7900 1300 30  0000 C CNN
+	1    7800 1300
 	0    -1   -1   0
 $EndComp
@@
 L TLV61220 U?
 U 1 1 504D3229
-P 9300 2600
-F 0 "U?" H 9250 2200 60  0000 C CNN
-F 1 "TLV61220" H 9300 2450 60  0000 C CNN
-	1    9300 2600
-	1    0    0    -1
-$EndComp
+P 9000 1600
+F 0 "U?" H 8950 1200 60  0000 C CNN
+F 1 "TLV61220" H 9000 1450 60  0000 C CNN
+	1    9000 1600
+	1    0    0    -1
+$EndComp
