File: pcb/power.sch (KiCad schematic (older format))
At the start: 22 parts, among them U2 LTC3559, U6 USBMICROCONN

Commit message: Added the 9V pin
Parts:
- added C?: 2.2n, symbol CAP
- added C?: 15p, symbol CAP
- added C?: 10u, symbol CAP
- added C?: 10n, symbol CAP
- added C?: 4.7u, symbol CAP
- added L?: CVH252009-4R7MCT-ND, symbol INDUCTOR
- added R?: 110k, symbol RES
- added R?: 18k, symbol RES
- added R?: 46.4k, symbol RES
- added R?: 10k, symbol RES
- added U?: LM4510, symbol LM4510
Connections:
- net labels added: POW_9V, Vnxt9v
- wire segments 78 -> 151

Commit message: Added voltage switching module.
Connections:
- net labels added: Vnxt4.3v
- net labels removed: Vnxt
Changed lines of the file:
@@
-EESchema Schematic File Version 2  date 9/10/2012 2:20:57 PM
+EESchema Schematic File Version 2  date 9/10/2012 3:24:02 PM
 LIBS:power
 LIBS:device
@@
 LIBS:valves
 LIBS:f4_daughter
+LIBS:f4_daughter-cache
 EELAYER 25  0
 EELAYER END
@@
 POW_NXT
 Text GLabel 10250 1600 2    60   Output ~ 0
-Vnxt
+Vnxt4.3v
 Text GLabel 7200 1100 0    60   Input ~ 0
 Vbat

Commit message: Adjusted the values of the pull down resistors.
Parts:
- R? (x2): value 10k -> 110k
Changed lines of the file:
@@
-EESchema Schematic File Version 2  date 9/10/2012 3:24:02 PM
+EESchema Schematic File Version 2  date 9/10/2012 5:54:09 PM
 LIBS:power
 LIBS:device
@@
 P 1950 5850
 F 0 "R?" H 2020 5815 30  0000 L TNN
-F 1 "10k" H 1950 5905 30  0000 C BNN
+F 1 "110k" H 1950 5905 30  0000 C BNN
 	1    1950 5850
 	0    -1   -1   0
@@
 P 8250 2100
 F 0 "R?" H 8320 2065 50  0000 L TNN
-F 1 "10k" H 8250 2155 30  0000 C BNN
+F 1 "110k" H 8250 2155 30  0000 C BNN
 	1    8250 2100
 	0    -1   -1   0

Commit message: Assigned lots of footprints, added diode footprint
Parts:
- gave numbers to parts that had none: 17
Connections:
- wire segments 151 -> 112

Commit message: Separated the NXT components from the main board. There were no real modifications in audio, rf or power, but kicad did modified some stuff that I wasn't sure so I committed everything just in case.
Connections:
- net labels added: EN_POW_NXT
- net labels removed: POW_NXT
Changed lines of the file:
@@
-EESchema Schematic File Version 2  date Wed 26 Sep 2012 06:41:48 PM EDT
+EESchema Schematic File Version 2  date 10/8/2012 8:27:48 PM
 LIBS:power
 LIBS:device
@@
 $Descr A4 11700 8267
 encoding utf-8
-Sheet 5 6
+Sheet 6 7
 Title ""
-Date "26 sep 2012"
+Date "9 oct 2012"
 Rev ""
 Comp ""
@@
 Connection ~ 1950 5450
 $Comp
-L GND #PWR027
+L GND #PWR27
 U 1 1 504E28B4
 P 1550 5900
-F 0 "#PWR027" H 1550 5900 30  0001 C CNN
+F 0 "#PWR27" H 1550 5900 30  0001 C CNN
 F 1 "GND" H 1550 5830 30  0001 C CNN
 	1    1550 5900
@@
 Vbat
 $Comp
-L GND #PWR028
+L GND #PWR30
 U 1 1 504E231C
 P 3200 6150
-F 0 "#PWR028" H 3200 6150 30  0001 C CNN
+F 0 "#PWR30" H 3200 6150 30  0001 C CNN
 F 1 "GND" H 3200 6080 30  0001 C CNN
 	1    3200 6150
@@
 $EndComp
 $Comp
-L GND #PWR029
+L GND #PWR28
 U 1 1 504E2309
 P 2100 5250
-F 0 "#PWR029" H 2100 5250 30  0001 C CNN
+F 0 "#PWR28" H 2100 5250 30  0001 C CNN
 F 1 "GND" H 2100 5180 30  0001 C CNN
 	1    2100 5250
@@
 $EndComp
 $Comp
-L GND #PWR030
+L GND #PWR37
 U 1 1 504E1CB3
 P 8250 2400
-F 0 "#PWR030" H 8250 2400 30  0001 C CNN
+F 0 "#PWR37" H 8250 2400 30  0001 C CNN
 F 1 "GND" H 8250 2330 30  0001 C CNN
 	1    8250 2400
@@
 $EndComp
 Text HLabel 8100 1900 0    60   Input ~ 0
-POW_NXT
+EN_POW_NXT
 Text GLabel 10250 1600 2    60   Output ~ 0
 Vnxt4.3v
@@
 Vbat
 $Comp
-L GND #PWR031
+L GND #PWR39
 U 1 1 504D34F8
 P 10050 2000
-F 0 "#PWR031" H 10050 2000 30  0001 C CNN
+F 0 "#PWR39" H 10050 2000 30  0001 C CNN
 F 1 "GND" H 10050 1930 30  0001 C CNN
 	1    10050 2000
@@
 $EndComp
 $Comp
-L GND #PWR032
+L GND #PWR38
 U 1 1 504D341F
 P 9800 2450
-F 0 "#PWR032" H 9800 2450 30  0001 C CNN
+F 0 "#PWR38" H 9800 2450 30  0001 C CNN
 F 1 "GND" H 9800 2380 30  0001 C CNN
 	1    9800 2450
@@
 $EndComp
 $Comp
-L GND #PWR033
+L GND #PWR36
 U 1 1 504D3361
 P 7400 1800
-F 0 "#PWR033" H 7400 1800 30  0001 C CNN
+F 0 "#PWR36" H 7400 1800 30  0001 C CNN
 F 1 "GND" H 7400 1730 30  0001 C CNN
 	1    7400 1800
@@
 $EndComp
 $Comp
-L GND #PWR034
+L GND #PWR33
 U 1 1 50117654
 P 5800 4150
-F 0 "#PWR034" H 5800 4150 30  0001 C CNN
+F 0 "#PWR33" H 5800 4150 30  0001 C CNN
 F 1 "GND" H 5800 4080 30  0001 C CNN
 	1    5800 4150
@@
 Vbus
 $Comp
-L GND #PWR035
+L GND #PWR35
 U 1 1 50116DE1
 P 6100 2100
-F 0 "#PWR035" H 6100 2100 30  0001 C CNN
+F 0 "#PWR35" H 6100 2100 30  0001 C CNN
 F 1 "GND" H 6100 2030 30  0001 C CNN
 	1    6100 2100
@@
 Vfb
 $Comp
-L GND #PWR036
+L GND #PWR32
 U 1 1 50116D88
 P 4250 4150
-F 0 "#PWR036" H 4250 4150 30  0001 C CNN
+F 0 "#PWR32" H 4250 4150 30  0001 C CNN
 F 1 "GND" H 4250 4080 30  0001 C CNN
 	1    4250 4150
@@
 Vbat
 $Comp
-L GND #PWR037
+L GND #PWR34
 U 1 1 50116D38
 P 6050 2950
-F 0 "#PWR037" H 6050 2950 30  0001 C CNN
+F 0 "#PWR34" H 6050 2950 30  0001 C CNN
 F 1 "GND" H 6050 2880 30  0001 C CNN
 	1    6050 2950
@@
 $EndComp
 $Comp
-L GND #PWR038
+L GND #PWR31
 U 1 1 50116D32
 P 4250 2500
-F 0 "#PWR038" H 4250 2500 30  0001 C CNN
+F 0 "#PWR31" H 4250 2500 30  0001 C CNN
 F 1 "GND" H 4250 2430 30  0001 C CNN
 	1    4250 2500
@@
 Vbus
 $Comp
-L GND #PWR039
+L GND #PWR29
 U 1 1 501093EE
 P 2700 2650
-F 0 "#PWR039" H 2700 2650 30  0001 C CNN
+F 0 "#PWR29" H 2700 2650 30  0001 C CNN
 F 1 "GND" H 2700 2580 30  0001 C CNN
 	1    2700 2650

Commit message: Reannoted everything so that there isn't any duplicates. Also added connection to the rf reset line.
Parts:
- renumbered C33 to C23, C34 to C24, C35 to C25, C1 to C26, C36 to C27, C37 to C28, C2 to C29, C3 to C30, C4 to C31, C5 to C32, C6 to C33, C38 to C34, C39 to C35, L3 to L2, L1 to L3, L2 to L4, R9 to R14, R21 to R15, R22 to R16, R23 to R17, R16 to R18, R17 to R19, R18 to R20, R19 to R21, R20 to R22, R24 to R23, R25 to R24, R26 to R25, U11 to U10, U6 to U7, U10 to U8, U2 to U9
Connections:
- net labels added: EN_POW_9V
- net labels removed: POW_9V

Commit message: A few more things: Added low-voltage battery detection to disable regulators Fixed XTAL symbol Annotated new components from yesterday
Parts:
- added R35: 680k, symbol RES
- added U13: MCP111T-315, symbol LV_DETECT
Connections:
- net labels added: REG_EN
- wire segments 112 -> 118
Changed lines of the file:
@@
-EESchema Schematic File Version 2  date 10/11/2012 11:52:24 AM
+EESchema Schematic File Version 2  date Sun 28 Oct 2012 01:53:13 PM EDT
 LIBS:power
 LIBS:device
@@
 Sheet 6 7
 Title ""
-Date "11 oct 2012"
+Date "28 oct 2012"
 Rev ""
 Comp ""
@@
 Comment4 ""
 $EndDescr
+Text Label 5200 3150 2    60   ~ 0
+REG_EN
+Text Label 3500 3550 2    60   ~ 0
+REG_EN
+Wire Wire Line
+	3100 3550 3500 3550
+Wire Wire Line
+	3500 3550 3500 3400
+Wire Wire Line
+	2850 4100 2850 3900
 Wire Wire Line
 	1550 5900 1550 5750
@@
 Connection ~ 3650 5150
 Wire Wire Line
-	3800 5150 2900 5150
+	2900 5150 3800 5150
 Wire Wire Line
 	2100 5750 2100 5550
@@
 Connection ~ 3450 5150
 Wire Wire Line
-	3650 5550 3650 5150
+	3650 5150 3650 5550
 Connection ~ 3100 5450
 Wire Wire Line
@@
 	3200 6100 3200 6150
 Wire Wire Line
-	3450 5150 3450 5200
+	3450 5200 3450 5150
 Wire Wire Line
 	2200 5250 2100 5250
@@
 	8250 1950 8250 1900
 Wire Wire Line
-	8100 1900 8400 1900
+	8400 1900 8100 1900
 Wire Wire Line
 	8400 1600 7400 1600
@@
 Connection ~ 3800 2650
 Wire Wire Line
-	3650 2650 4900 2650
+	4900 2650 3650 2650
 Wire Wire Line
 	3800 2950 3800 2650
@@
 	5450 1850 5450 2100
 Wire Wire Line
-	4250 4150 4250 3800
+	4250 3800 4250 4150
 Wire Wire Line
 	4250 3100 4250 3050
@@
 	4250 3050 4450 3050
 Wire Wire Line
-	4700 3350 4450 3350
+	4450 3350 4700 3350
 Wire Wire Line
 	5250 3100 5250 3150
@@
 	5350 3350 5350 3100
 Wire Wire Line
-	4250 3500 4250 3400
+	4250 3400 4250 3500
 Wire Wire Line
 	4250 3450 4050 3450
@@
 Connection ~ 4350 2750
 Wire Wire Line
-	4650 3500 4650 3150
-Wire Wire Line
-	5450 3400 5450 3100
+	4650 3150 4650 3500
+Wire Wire Line
+	5450 3100 5450 3400
 Wire Wire Line
 	2700 2650 2700 2500
@@
 	10050 2000 10050 1850
 Wire Wire Line
-	9600 1600 10250 1600
+	10250 1600 9600 1600
 Connection ~ 10050 1600
 Wire Wire Line
@@
 	3350 5550 3450 5550
 Wire Wire Line
-	3450 5500 3450 5600
+	3450 5600 3450 5500
 Connection ~ 3450 5550
 Wire Wire Line
@@
 	1800 5450 2200 5450
 Connection ~ 1950 5450
-$Comp
-L GND #PWR31
+Wire Wire Line
+	2850 3000 2850 3200
+Wire Wire Line
+	3500 3100 3500 3000
+Wire Wire Line
+	3500 3000 2750 3000
+Connection ~ 2850 3000
+$Comp
+L RES R35
+U 1 1 508D6BDD
+P 3500 3250
+F 0 "R35" H 3570 3215 50  0000 L TNN
+F 1 "680k" H 3500 3305 30  0000 C BNN
+	1    3500 3250
+	0    -1   -1   0
+$EndComp
+$Comp
+L GND #PWR35
+U 1 1 508D6B9D
+P 2850 4100
+F 0 "#PWR35" H 2850 4100 30  0001 C CNN
+F 1 "GND" H 2850 4030 30  0001 C CNN
+	1    2850 4100
+	1    0    0    -1
+$EndComp
+Text GLabel 2750 3000 0    60   Input ~ 0
+Vbat
+$Comp
+L LV_DETECT U13
+U 1 1 508D6B78
+P 2850 3550
+F 0 "U13" H 2950 3250 60  0000 C CNN
+F 1 "MCP111T-315" V 2650 3550 60  0000 C CNN
+	1    2850 3550
+	1    0    0    -1
+$EndComp
+$Comp
+L GND #PWR32
 U 1 1 504E28B4
 P 1550 5900
-F 0 "#PWR31" H 1550 5900 30  0001 C CNN
+F 0 "#PWR32" H 1550 5900 30  0001 C CNN
 F 1 "GND" H 1550 5830 30  0001 C CNN
 	1    1550 5900
@@
 Vbat
 $Comp
-L GND #PWR34
+L GND #PWR36
 U 1 1 504E231C
 P 3200 6150
-F 0 "#PWR34" H 3200 6150 30  0001 C CNN
+F 0 "#PWR36" H 3200 6150 30  0001 C CNN
 F 1 "GND" H 3200 6080 30  0001 C CNN
 	1    3200 6150
@@
 $EndComp
 $Comp
-L GND #PWR32
+L GND #PWR33
 U 1 1 504E2309
 P 2100 5250
-F 0 "#PWR32" H 2100 5250 30  0001 C CNN
+F 0 "#PWR33" H 2100 5250 30  0001 C CNN
 F 1 "GND" H 2100 5180 30  0001 C CNN
 	1    2100 5250
@@
 $EndComp
 $Comp
-L GND #PWR41
+L GND #PWR43
 U 1 1 504E1CB3
 P 8250 2400
-F 0 "#PWR41" H 8250 2400 30  0001 C CNN
+F 0 "#PWR43" H 8250 2400 30  0001 C CNN
 F 1 "GND" H 8250 2330 30  0001 C CNN
 	1    8250 2400
@@
 Vbat
 $Comp
-L GND #PWR43
+L GND #PWR45
 U 1 1 504D34F8
 P 10050 2000
-F 0 "#PWR43" H 10050 2000 30  0001 C CNN
+F 0 "#PWR45" H 10050 2000 30  0001 C CNN
 F 1 "GND" H 10050 1930 30  0001 C CNN
 	1    10050 2000
@@
 $EndComp
 $Comp
-L GND #PWR42
+L GND #PWR44
 U 1 1 504D341F
 P 9800 2450
-F 0 "#PWR42" H 9800 2450 30  0001 C CNN
+F 0 "#PWR44" H 9800 2450 30  0001 C CNN
 F 1 "GND" H 9800 2380 30  0001 C CNN
 	1    9800 2450
@@
 $EndComp
 $Comp
-L GND #PWR40
+L GND #PWR42
 U 1 1 504D3361
 P 7400 1800
-F 0 "#PWR40" H 7400 1800 30  0001 C CNN
+F 0 "#PWR42" H 7400 1800 30  0001 C CNN
 F 1 "GND" H 7400 1730 30  0001 C CNN
 	1    7400 1800
@@
 $EndComp
 $Comp
-L GND #PWR37
+L GND #PWR39
 U 1 1 50117654
 P 5800 4150
-F 0 "#PWR37" H 5800 4150 30  0001 C CNN
+F 0 "#PWR39" H 5800 4150 30  0001 C CNN
 F 1 "GND" H 5800 4080 30  0001 C CNN
 	1    5800 4150
@@
 Vbus
 $Comp
-L GND #PWR39
+L GND #PWR41
 U 1 1 50116DE1
 P 6100 2100
-F 0 "#PWR39" H 6100 2100 30  0001 C CNN
+F 0 "#PWR41" H 6100 2100 30  0001 C CNN
 F 1 "GND" H 6100 2030 30  0001 C CNN
 	1    6100 2100
@@
 Vfb
 $Comp
-L GND #PWR36
+L GND #PWR38
 U 1 1 50116D88
 P 4250 4150
-F 0 "#PWR36" H 4250 4150 30  0001 C CNN
+F 0 "#PWR38" H 4250 4150 30  0001 C CNN
 F 1 "GND" H 4250 4080 30  0001 C CNN
 	1    4250 4150
@@
 	0    -1   -1   0
 $EndComp
-Text GLabel 5200 3150 0    60   Input ~ 0
-Vbat
-$Comp
-L GND #PWR38
+$Comp
+L GND #PWR40
 U 1 1 50116D38
 P 6050 2950
-F 0 "#PWR38" H 6050 2950 30  0001 C CNN
+F 0 "#PWR40" H 6050 2950 30  0001 C CNN
 F 1 "GND" H 6050 2880 30  0001 C CNN
 	1    6050 2950
@@
 $EndComp
 $Comp
-L GND #PWR35
+L GND #PWR37
 U 1 1 50116D32
 P 4250 2500
-F 0 "#PWR35" H 4250 2500 30  0001 C CNN
+F 0 "#PWR37" H 4250 2500 30  0001 C CNN
 F 1 "GND" H 4250 2430 30  0001 C CNN
 	1    4250 2500
@@
 Vbus
 $Comp
-L GND #PWR33
+L GND #PWR34
 U 1 1 501093EE
 P 2700 2650
-F 0 "#PWR33" H 2700 2650 30  0001 C CNN
+F 0 "#PWR34" H 2700 2650 30  0001 C CNN
 F 1 "GND" H 2700 2580 30  0001 C CNN
 	1    2700 2650
