File: pcb/power.sch (KiCad schematic (older format))
At the start: 35 parts, among them U10 TLV61220, U13 MCP111T-315, U7 USBMICROCONN, U8 LM4510, U9 LTC3559

Commit message: Changed some values and connected more LCD signals
Parts:
- C24: value 10n -> 0.01u
- C26: value 10u -> 2.2u
- C31: value 470n -> 0.47u
Connections:
- wire segments 118 -> 122
Other:
- moved on the sheet: C34, C35, R15, R23, R24, R25

Commit message: Adjusted 3V regulator voltage divider
Parts:
- R19: value 220k(1%) -> 604k(1%)
- R20: value 680k(1%) -> 220k(1%)
Changed lines of the file:
@@
-EESchema Schematic File Version 2  date Sun 28 Oct 2012 06:31:28 PM EDT
+EESchema Schematic File Version 2  date Thu 01 Nov 2012 03:50:31 PM EDT
 LIBS:power
 LIBS:device
@@
 Sheet 6 7
 Title ""
-Date "28 oct 2012"
+Date "1 nov 2012"
 Rev ""
 Comp ""
@@
 P 4250 3650
 F 0 "R20" H 4320 3615 50  0000 L TNN
-F 1 "680k(1%)" H 4250 3705 30  0000 C BNN
+F 1 "220k(1%)" H 4250 3705 30  0000 C BNN
 	1    4250 3650
 	0    -1   -1   0
@@
 P 4250 3250
 F 0 "R19" H 4320 3215 50  0000 L TNN
-F 1 "220k(1%)" H 4250 3305 30  0000 C BNN
+F 1 "604k(1%)" H 4250 3305 30  0000 C BNN
 	1    4250 3250
 	0    -1   -1   0

Commit message: Added CPLD, CPLD doc, and backlight driver doc
Parts:
- added C?: 0.1u, symbol CAP
- added C?: 2.2u, symbol CAP
- added C?: 22p, symbol CAP
- added L?: CVH252009-4R7MCT-ND, symbol INDUCTOR
- added R?: 560k(1%), symbol RES
- added R?: 720k(1%), symbol RES
- added R?: 220k, symbol RES
Connections:
- net labels added: CPLD_PWR_EN, V1.8
- wire segments 122 -> 140

Commit message: Added backlight driver, connected to I2C1, annotated stuff
Parts:
- gave numbers to parts that had none: 7
Changed lines of the file:
@@
-EESchema Schematic File Version 2  date 12/19/2012 4:02:29 PM
+EESchema Schematic File Version 2  date Fri 28 Dec 2012 12:18:10 AM EST
 LIBS:power
 LIBS:device
@@
 Sheet 8 9
 Title ""
-Date "19 dec 2012"
+Date "28 dec 2012"
 Rev ""
 Comp ""
@@
 V1.8
 $Comp
-L RES R?
+L RES R41
 U 1 1 50C0E98E
 P 7550 3500
-F 0 "R?" H 7620 3465 50  0000 L TNN
+F 0 "R41" H 7620 3465 50  0000 L TNN
 F 1 "220k" H 7550 3555 30  0000 C BNN
 	1    7550 3500
@@
 $EndComp
 $Comp
-L CAP C?
+L CAP C48
 U 1 1 50C0CDF3
 P 7150 2950
-F 0 "C?" H 7170 2920 50  0000 L TNN
+F 0 "C48" H 7170 2920 50  0000 L TNN
 F 1 "22p" H 7175 2970 30  0000 L BNN
 	1    7150 2950
@@
 CPLD_PWR_EN
 $Comp
-L GND #PWR?
+L GND #PWR46
 U 1 1 50C0C86E
 P 7000 4200
-F 0 "#PWR?" H 7000 4200 30  0001 C CNN
+F 0 "#PWR46" H 7000 4200 30  0001 C CNN
 F 1 "GND" H 7000 4130 30  0001 C CNN
 	1    7000 4200
@@
 $EndComp
 $Comp
-L CAP C?
+L CAP C47
 U 1 1 50C0C850
 P 7000 3650
-F 0 "C?" H 7020 3620 50  0000 L TNN
+F 0 "C47" H 7020 3620 50  0000 L TNN
 F 1 "2.2u" H 7025 3670 30  0000 L BNN
 	1    7000 3650
@@
 $EndComp
 $Comp
-L CAP C?
+L CAP C46
 U 1 1 50C0C84C
 P 6850 3650
-F 0 "C?" H 6870 3620 50  0000 L TNN
+F 0 "C46" H 6870 3620 50  0000 L TNN
 F 1 "0.1u" H 6875 3670 30  0000 L BNN
 	1    6850 3650
@@
 $EndComp
 $Comp
-L INDUCTOR L?
+L INDUCTOR L6
 U 1 1 50C0C836
 P 6450 3200
-F 0 "L?" V 6400 3200 40  0000 C CNN
+F 0 "L6" V 6400 3200 40  0000 C CNN
 F 1 "CVH252009-4R7MCT-ND" V 6550 3200 30  0000 C CNN
 	1    6450 3200
@@
 $EndComp
 $Comp
-L RES R?
+L RES R39
 U 1 1 50C0C824
 P 7250 3450
-F 0 "R?" H 7320 3415 50  0000 L TNN
+F 0 "R39" H 7320 3415 50  0000 L TNN
 F 1 "720k(1%)" H 7250 3505 30  0000 C BNN
 	1    7250 3450
@@
 $EndComp
 $Comp
-L RES R?
+L RES R40
 U 1 1 50C0C823
 P 7250 3850
-F 0 "R?" H 7320 3815 50  0000 L TNN
+F 0 "R40" H 7320 3815 50  0000 L TNN
 F 1 "560k(1%)" H 7250 3905 30  0000 C BNN
 	1    7250 3850
@@
 $EndComp
 $Comp
-L GND #PWR35
+L GND #PWR39
 U 1 1 508D6B9D
 P 2850 4100
-F 0 "#PWR35" H 2850 4100 30  0001 C CNN
+F 0 "#PWR39" H 2850 4100 30  0001 C CNN
 F 1 "GND" H 2850 4030 30  0001 C CNN
 	1    2850 4100
@@
 $EndComp
 $Comp
-L GND #PWR32
+L GND #PWR36
 U 1 1 504E28B4
 P 1550 5900
-F 0 "#PWR32" H 1550 5900 30  0001 C CNN
+F 0 "#PWR36" H 1550 5900 30  0001 C CNN
 F 1 "GND" H 1550 5830 30  0001 C CNN
 	1    1550 5900
@@
 Vbat
 $Comp
-L GND #PWR36
+L GND #PWR40
 U 1 1 504E231C
 P 3200 6150
-F 0 "#PWR36" H 3200 6150 30  0001 C CNN
+F 0 "#PWR40" H 3200 6150 30  0001 C CNN
 F 1 "GND" H 3200 6080 30  0001 C CNN
 	1    3200 6150
@@
 $EndComp
 $Comp
-L GND #PWR33
+L GND #PWR37
 U 1 1 504E2309
 P 2100 5250
-F 0 "#PWR33" H 2100 5250 30  0001 C CNN
+F 0 "#PWR37" H 2100 5250 30  0001 C CNN
 F 1 "GND" H 2100 5180 30  0001 C CNN
 	1    2100 5250
@@
 $EndComp
 $Comp
-L GND #PWR43
+L GND #PWR48
 U 1 1 504E1CB3
 P 8250 2400
-F 0 "#PWR43" H 8250 2400 30  0001 C CNN
+F 0 "#PWR48" H 8250 2400 30  0001 C CNN
 F 1 "GND" H 8250 2330 30  0001 C CNN
 	1    8250 2400
@@
 Vbat
 $Comp
-L GND #PWR45
+L GND #PWR50
 U 1 1 504D34F8
 P 10050 2000
-F 0 "#PWR45" H 10050 2000 30  0001 C CNN
+F 0 "#PWR50" H 10050 2000 30  0001 C CNN
 F 1 "GND" H 10050 1930 30  0001 C CNN
 	1    10050 2000
@@
 $EndComp
 $Comp
-L GND #PWR44
+L GND #PWR49
 U 1 1 504D341F
 P 9800 2450
-F 0 "#PWR44" H 9800 2450 30  0001 C CNN
+F 0 "#PWR49" H 9800 2450 30  0001 C CNN
 F 1 "GND" H 9800 2380 30  0001 C CNN
 	1    9800 2450
@@
 $EndComp
 $Comp
-L GND #PWR42
+L GND #PWR47
 U 1 1 504D3361
 P 7400 1800
-F 0 "#PWR42" H 7400 1800 30  0001 C CNN
+F 0 "#PWR47" H 7400 1800 30  0001 C CNN
 F 1 "GND" H 7400 1730 30  0001 C CNN
 	1    7400 1800
@@
 $EndComp
 $Comp
-L GND #PWR39
+L GND #PWR43
 U 1 1 50117654
 P 5800 4150
-F 0 "#PWR39" H 5800 4150 30  0001 C CNN
+F 0 "#PWR43" H 5800 4150 30  0001 C CNN
 F 1 "GND" H 5800 4080 30  0001 C CNN
 	1    5800 4150
@@
 Vbus
 $Comp
-L GND #PWR41
+L GND #PWR45
 U 1 1 50116DE1
 P 6100 2100
-F 0 "#PWR41" H 6100 2100 30  0001 C CNN
+F 0 "#PWR45" H 6100 2100 30  0001 C CNN
 F 1 "GND" H 6100 2030 30  0001 C CNN
 	1    6100 2100
@@
 Vfb
 $Comp
-L GND #PWR38
+L GND #PWR42
 U 1 1 50116D88
 P 4250 4150
-F 0 "#PWR38" H 4250 4150 30  0001 C CNN
+F 0 "#PWR42" H 4250 4150 30  0001 C CNN
 F 1 "GND" H 4250 4080 30  0001 C CNN
 	1    4250 4150
@@
 $EndComp
 $Comp
-L GND #PWR40
+L GND #PWR44
 U 1 1 50116D38
 P 6050 2950
-F 0 "#PWR40" H 6050 2950 30  0001 C CNN
+F 0 "#PWR44" H 6050 2950 30  0001 C CNN
 F 1 "GND" H 6050 2880 30  0001 C CNN
 	1    6050 2950
@@
 $EndComp
 $Comp
-L GND #PWR37
+L GND #PWR41
 U 1 1 50116D32
 P 4250 2500
-F 0 "#PWR37" H 4250 2500 30  0001 C CNN
+F 0 "#PWR41" H 4250 2500 30  0001 C CNN
 F 1 "GND" H 4250 2430 30  0001 C CNN
 	1    4250 2500
@@
 Vbus
 $Comp
-L GND #PWR34
+L GND #PWR38
 U 1 1 501093EE
 P 2700 2650
-F 0 "#PWR34" H 2700 2650 30  0001 C CNN
+F 0 "#PWR38" H 2700 2650 30  0001 C CNN
 F 1 "GND" H 2700 2580 30  0001 C CNN
 	1    2700 2650
