File: pcb/audio_in.sch (KiCad schematic (older format))
At the start: 17 parts, among them J2 SJ1-3523N, U7 MCP6409

Commit message: Better audio filters
Parts:
- removed R6, R9: 100k(1%), symbol RES
- added C?: 100n, symbol CAP
- added R? (x2): 100k, symbol TRIM_R
- added unit 4 of U7
- added U?: MCP6241, symbol OPAMP
Connections:
- wire segments 55 -> 89
Other:
- moved on the sheet: C26, C27, C28, C29, C30, C31, C7, R10, R11, R12, R13, R14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

Commit message: Assigned lots of footprints, added diode footprint
Parts:
- gave numbers to parts that had none: 4
Connections:
- wire segments 89 -> 73
Changed lines of the file:
@@
-EESchema Schematic File Version 2  date Fri 07 Sep 2012 05:49:39 PM EDT
+EESchema Schematic File Version 2  date Wed 26 Sep 2012 06:41:48 PM EDT
 LIBS:power
 LIBS:device
@@
 Sheet 6 6
 Title ""
-Date "7 sep 2012"
+Date "26 sep 2012"
 Rev ""
 Comp ""
@@
 	2200 2900 2300 2900
 Wire Wire Line
-	2800 2800 3000 2800
-Wire Wire Line
-	3000 2800 3200 2800
+	2800 2800 3200 2800
 Wire Wire Line
 	1650 3800 1900 3800
@@
 Connection ~ 8950 5000
 Wire Wire Line
-	9150 5000 8950 5000
-Wire Wire Line
-	8950 5000 8800 5000
+	9150 5000 8800 5000
 Wire Wire Line
 	8950 5000 8950 5350
@@
 	8200 5100 8300 5100
 Wire Wire Line
-	7700 4500 7700 4450
-Wire Wire Line
-	7700 4450 7700 4400
+	7700 4500 7700 4400
 Connection ~ 5150 4200
 Wire Wire Line
-	5300 4200 5150 4200
-Wire Wire Line
-	5150 4200 4900 4200
-Wire Wire Line
-	5150 4550 5150 4200
-Wire Wire Line
-	5150 4200 5150 3800
+	5300 4200 4900 4200
+Wire Wire Line
+	5150 4550 5150 3800
 Wire Wire Line
 	5150 4550 4350 4550
@@
 	4350 4300 4450 4300
 Wire Wire Line
-	7700 5400 7700 5350
-Wire Wire Line
-	7700 5350 7700 5300
+	7700 5400 7700 5300
 Connection ~ 3550 4100
 Wire Wire Line
-	3600 4100 3550 4100
-Wire Wire Line
-	3550 4100 3450 4100
+	3600 4100 3450 4100
 Connection ~ 4100 4100
 Wire Wire Line
 	4100 4250 4100 4100
 Wire Wire Line
-	4450 4100 4100 4100
-Wire Wire Line
-	4100 4100 3900 4100
+	4450 4100 3900 4100
 Wire Wire Line
 	5150 3800 4350 3800
@@
 Connection ~ 7700 4900
 Wire Wire Line
-	8300 4900 7950 4900
-Wire Wire Line
-	7950 4900 7700 4900
-Wire Wire Line
-	7700 5000 7700 4900
-Wire Wire Line
-	7700 4900 7700 4800
+	8300 4900 7700 4900
+Wire Wire Line
+	7700 5000 7700 4800
 Connection ~ 5150 2900
 Wire Wire Line
@@
 Connection ~ 3550 2800
 Wire Wire Line
-	3600 2800 3550 2800
-Wire Wire Line
-	3550 2800 3500 2800
+	3600 2800 3500 2800
 Connection ~ 4100 2800
 Wire Wire Line
 	4100 2950 4100 2800
 Wire Wire Line
-	4450 2800 4100 2800
-Wire Wire Line
-	4100 2800 3900 2800
-Wire Wire Line
-	5350 2900 5150 2900
-Wire Wire Line
-	5150 2900 4950 2900
-Wire Wire Line
-	5150 3250 5150 2900
-Wire Wire Line
-	5150 2900 5150 2500
+	4450 2800 3900 2800
+Wire Wire Line
+	5350 2900 4950 2900
+Wire Wire Line
+	5150 3250 5150 2500
 Wire Wire Line
 	5150 2500 4350 2500
@@
 	3550 2500 3550 2800
 Wire Wire Line
-	6750 6100 6750 6150
-Wire Wire Line
-	6750 6150 6750 6250
+	6750 6100 6750 6250
 Wire Wire Line
 	6750 5550 6750 5450
@@
 	1900 2850 1900 3050
 Wire Wire Line
-	2800 4100 3000 4100
-Wire Wire Line
-	3000 4100 3150 4100
+	2800 4100 3150 4100
 Wire Wire Line
 	2300 2700 2050 2700
@@
 Connection ~ 7950 4900
 $Comp
-L CAP C?
+L CAP C40
 U 1 1 504649FC
 P 7950 5150
-F 0 "C?" H 7970 5120 50  0000 L TNN
+F 0 "C40" H 7970 5120 50  0000 L TNN
 F 1 "100n" H 7975 5170 30  0000 L BNN
 	1    7950 5150
@@
 $EndComp
 $Comp
-L GND #PWR?
+L GND #PWR040
 U 1 1 504649EC
 P 8550 5250
-F 0 "#PWR?" H 8550 5250 30  0001 C CNN
+F 0 "#PWR040" H 8550 5250 30  0001 C CNN
 F 1 "GND" H 8550 5180 30  0001 C CNN
 	1    8550 5250
@@
 $EndComp
 $Comp
-L OPAMP U?
+L OPAMP U12
 U 1 1 504649E3
 P 8500 5000
-F 0 "U?" H 8650 4850 60  0000 C CNN
+F 0 "U12" H 8650 4850 60  0000 C CNN
 F 1 "MCP6241" H 8750 5150 60  0000 C CNN
 F 3 "http://ww1.microchip.com/downloads/en/DeviceDoc/21882d.pdf" H 8500 5000 60  0001 C CNN
@@
 $EndComp
 $Comp
-L TRIM_R R?
+L TRIM_R R28
 U 1 1 504632BD
 P 1900 4000
-F 0 "R?" H 1970 3965 50  0000 L TNN
+F 0 "R28" H 1970 3965 50  0000 L TNN
 F 1 "100k" H 1900 4055 30  0000 C BNN
 	1    1900 4000
@@
 $EndComp
 $Comp
-L TRIM_R R?
+L TRIM_R R27
 U 1 1 5046327E
 P 1900 2700
-F 0 "R?" H 1970 2665 50  0000 L TNN
+F 0 "R27" H 1970 2665 50  0000 L TNN
 F 1 "100k" H 1900 2755 30  0000 C BNN
 	1    1900 2700
@@
 VGND
 $Comp
-L GND #PWR027
+L GND #PWR041
 U 1 1 50118BD6
 P 1050 3000
-F 0 "#PWR027" H 1050 3000 30  0001 C CNN
+F 0 "#PWR041" H 1050 3000 30  0001 C CNN
 F 1 "GND" H 1050 2930 30  0001 C CNN
 	1    1050 3000
@@
 Vreg
 $Comp
-L GND #PWR028
+L GND #PWR042
 U 1 1 5010D90D
 P 6750 6250
-F 0 "#PWR028" H 6750 6250 30  0001 C CNN
+F 0 "#PWR042" H 6750 6250 30  0001 C CNN
 F 1 "GND" H 6750 6180 30  0001 C CNN
 	1    6750 6250
@@
 Vreg
 $Comp
-L GND #PWR029
+L GND #PWR043
 U 1 1 5010DA28
 P 7700 5400
-F 0 "#PWR029" H 7700 5400 30  0001 C CNN
+F 0 "#PWR043" H 7700 5400 30  0001 C CNN
 F 1 "GND" H 7700 5330 30  0001 C CNN
 	1    7700 5400

Commit message: Reannoted everything so that there isn't any duplicates. Also added connection to the rf reset line.
Parts:
- renumbered C31 to C36, C30 to C37, C26 to C38, C27 to C39, C28 to C40, C29 to C41, C7 to C42, C40 to C43, J2 to J5, R27 to R26, R28 to R27, R11 to R28, R10 to R29, R12 to R30, R13 to R31, R14 to R32, R15 to R33, U7 to U11
Changed lines of the file:
@@
-EESchema Schematic File Version 2  date 10/10/2012 1:41:54 PM
+EESchema Schematic File Version 2  date 10/11/2012 11:52:24 AM
 LIBS:power
 LIBS:device
@@
 Sheet 7 7
 Title ""
-Date "10 oct 2012"
+Date "11 oct 2012"
 Rev ""
 Comp ""
@@
 Connection ~ 7950 4900
 $Comp
-L CAP C40
+L CAP C43
 U 1 1 504649FC
 P 7950 5150
-F 0 "C40" H 7970 5120 50  0000 L TNN
+F 0 "C43" H 7970 5120 50  0000 L TNN
 F 1 "100n" H 7975 5170 30  0000 L BNN
 	1    7950 5150
@@
 $EndComp
 $Comp
-L GND #PWR45
+L GND #PWR47
 U 1 1 504649EC
 P 8550 5250
-F 0 "#PWR45" H 8550 5250 30  0001 C CNN
+F 0 "#PWR47" H 8550 5250 30  0001 C CNN
 F 1 "GND" H 8550 5180 30  0001 C CNN
 	1    8550 5250
@@
 $EndComp
 $Comp
-L MCP6409 U7
-U 4 1 50464816
+L MCP6409 U11
+U 1 1 50464816
 P 2500 2800
-F 0 "U7" H 2600 2500 60  0000 C CNN
+F 0 "U11" H 2600 2500 60  0000 C CNN
 F 1 "MCP6409" H 2750 2950 60  0000 C CNN
-	4    2500 2800
-	1    0    0    -1
-$EndComp
-$Comp
-L TRIM_R R28
+	1    2500 2800
+	1    0    0    -1
+$EndComp
+$Comp
+L TRIM_R R27
 U 1 1 504632BD
 P 1900 4000
-F 0 "R28" H 1970 3965 50  0000 L TNN
+F 0 "R27" H 1970 3965 50  0000 L TNN
 F 1 "100k" H 1900 4055 30  0000 C BNN
 	1    1900 4000
@@
 $EndComp
 $Comp
-L TRIM_R R27
+L TRIM_R R26
 U 1 1 5046327E
 P 1900 2700
-F 0 "R27" H 1970 2665 50  0000 L TNN
+F 0 "R26" H 1970 2665 50  0000 L TNN
 F 1 "100k" H 1900 2755 30  0000 C BNN
 	1    1900 2700
@@
 VGND
 $Comp
-L GND #PWR42
+L GND #PWR44
 U 1 1 50118BD6
 P 1050 3000
-F 0 "#PWR42" H 1050 3000 30  0001 C CNN
+F 0 "#PWR44" H 1050 3000 30  0001 C CNN
 F 1 "GND" H 1050 2930 30  0001 C CNN
 	1    1050 3000
@@
 $EndComp
 $Comp
-L TRS_CONN J2
+L TRS_CONN J5
 U 1 1 50118BBE
 P 800 3350
-F 0 "J2" H 1100 3100 60  0000 C CNN
+F 0 "J5" H 1100 3100 60  0000 C CNN
 F 1 "SJ1-3523N" H 750 3600 60  0000 C CNN
 	1    800  3350
@@
 $EndComp
 $Comp
-L CAP C7
+L CAP C42
 U 1 1 50118878
 P 7000 5800
-F 0 "C7" H 7020 5770 50  0000 L TNN
+F 0 "C42" H 7020 5770 50  0000 L TNN
 F 1 "100n" H 7025 5820 30  0000 L BNN
 	1    7000 5800
@@
 $EndComp
 $Comp
-L MCP6409 U7
-U 1 1 5010D8C5
+L MCP6409 U11
+U 4 1 5010D8C5
 P 4650 2900
-F 0 "U7" H 4750 2600 60  0000 C CNN
+F 0 "U11" H 4750 2600 60  0000 C CNN
 F 1 "MCP6409" H 4900 3050 60  0000 C CNN
-	1    4650 2900
-	1    0    0    -1
-$EndComp
-$Comp
-L MCP6409 U7
-U 2 1 5010D8D4
+	4    4650 2900
+	1    0    0    -1
+$EndComp
+$Comp
+L MCP6409 U11
+U 3 1 5010D8D4
 P 4600 4200
-F 0 "U7" H 4700 3900 60  0000 C CNN
+F 0 "U11" H 4700 3900 60  0000 C CNN
 F 1 "MCP6409" H 4850 4350 60  0000 C CNN
-	2    4600 4200
-	1    0    0    -1
-$EndComp
-$Comp
-L MCP6409 U7
-U 3 1 5010D8E3
+	3    4600 4200
+	1    0    0    -1
+$EndComp
+$Comp
+L MCP6409 U11
+U 2 1 5010D8E3
 P 2500 4100
-F 0 "U7" H 2600 3800 60  0000 C CNN
+F 0 "U11" H 2600 3800 60  0000 C CNN
 F 1 "MCP6409" H 2750 4250 60  0000 C CNN
-	3    2500 4100
-	1    0    0    -1
-$EndComp
-$Comp
-L MCP6409 U7
+	2    2500 4100
+	1    0    0    -1
+$EndComp
+$Comp
+L MCP6409 U11
 U 5 1 5010D8F2
 P 6750 5750
-F 0 "U7" H 6850 5450 60  0000 C CNN
+F 0 "U11" H 6850 5450 60  0000 C CNN
 F 1 "MCP6409" H 6450 5900 60  0000 C CNN
 	5    6750 5750
@@
 Vreg
 $Comp
-L GND #PWR43
+L GND #PWR45
 U 1 1 5010D90D
 P 6750 6250
-F 0 "#PWR43" H 6750 6250 30  0001 C CNN
+F 0 "#PWR45" H 6750 6250 30  0001 C CNN
 F 1 "GND" H 6750 6180 30  0001 C CNN
 	1    6750 6250
@@
 $EndComp
 $Comp
-L RES R10
+L RES R29
 U 1 1 5010D91F
 P 3350 2800
-F 0 "R10" H 3420 2765 50  0000 L TNN
+F 0 "R29" H 3420 2765 50  0000 L TNN
 F 1 "2.8k(1%)" H 3350 2855 30  0000 C BNN
 	1    3350 2800
@@
 $EndComp
 $Comp
-L RES R12
+L RES R30
 U 1 1 5010D92C
 P 3750 2800
-F 0 "R12" H 3820 2765 50  0000 L TNN
+F 0 "R30" H 3820 2765 50  0000 L TNN
 F 1 "2.8k(1%)" H 3750 2855 30  0000 C BNN
 	1    3750 2800
@@
 $EndComp
 $Comp
-L CAP C26
+L CAP C38
 U 1 1 5010D940
 P 4100 3050
-F 0 "C26" H 4120 3020 50  0000 L TNN
+F 0 "C38" H 4120 3020 50  0000 L TNN
 F 1 "2.4n(5%)" H 4125 3070 30  0000 L BNN
 	1    4100 3050
@@
 $EndComp
 $Comp
-L CAP C28
+L CAP C40
 U 1 1 5010D94D
 P 4250 2500
-F 0 "C28" H 4270 2470 50  0000 L TNN
+F 0 "C40" H 4270 2470 50  0000 L TNN
 F 1 "4.7n(5%)" H 4275 2520 30  0000 L BNN
 	1    4250 2500
@@
 $EndComp
 $Comp
-L RES R13
+L RES R31
 U 1 1 5010D9FD
 P 3750 4100
-F 0 "R13" H 3820 4065 50  0000 L TNN
+F 0 "R31" H 3820 4065 50  0000 L TNN
 F 1 "2.8k(1%)" H 3750 4155 30  0000 C BNN
 	1    3750 4100
@@
 $EndComp
 $Comp
-L RES R14
+L RES R32
 U 1 1 5010DA03
 P 7700 4650
-F 0 "R14" H 7770 4615 50  0000 L TNN
+F 0 "R32" H 7770 4615 50  0000 L TNN
 F 1 "100k(1%)" H 7700 4705 30  0000 C BNN
 	1    7700 4650
@@
 $EndComp
 $Comp
-L RES R15
+L RES R33
 U 1 1 5010DA09
 P 7700 5150
-F 0 "R15" H 7770 5115 50  0000 L TNN
+F 0 "R33" H 7770 5115 50  0000 L TNN
 F 1 "100k(1%)" H 7700 5205 30  0000 C BNN
 	1    7700 5150
@@
 $EndComp
 $Comp
-L CAP C27
+L CAP C39
 U 1 1 5010DA0F
 P 4100 4350
-F 0 "C27" H 4120 4320 50  0000 L TNN
+F 0 "C39" H 4120 4320 50  0000 L TNN
 F 1 "2.4n(5%)" H 4125 4370 30  0000 L BNN
 	1    4100 4350
@@
 $EndComp
 $Comp
-L CAP C29
+L CAP C41
 U 1 1 5010DA15
 P 4250 3800
-F 0 "C29" H 4270 3770 50  0000 L TNN
+F 0 "C41" H 4270 3770 50  0000 L TNN
 F 1 "4.7n(5%)" H 4275 3820 30  0000 L BNN
 	1    4250 3800
@@
 Vreg
 $Comp
-L GND #PWR44
+L GND #PWR46
 U 1 1 5010DA28
 P 7700 5400
-F 0 "#PWR44" H 7700 5400 30  0001 C CNN
+F 0 "#PWR46" H 7700 5400 30  0001 C CNN
 F 1 "GND" H 7700 5330 30  0001 C CNN
 	1    7700 5400
@@
 VGND
 $Comp
-L RES R11
+L RES R28
 U 1 1 5010DC47
 P 3300 4100
-F 0 "R11" H 3370 4065 50  0000 L TNN
+F 0 "R28" H 3370 4065 50  0000 L TNN
 F 1 "2.8k(1%)" H 3300 4155 30  0000 C BNN
 	1    3300 4100
@@
 $EndComp
 $Comp
-L CAP C30
+L CAP C37
 U 1 1 5010E008
 P 1600 2500
-F 0 "C30" H 1620 2470 50  0000 L TNN
+F 0 "C37" H 1620 2470 50  0000 L TNN
 F 1 "0.47u" H 1625 2520 30  0000 L BNN
 	1    1600 2500
@@
 $EndComp
 $Comp
-L CAP C31
+L CAP C36
 U 1 1 5010E015
 P 1550 3800
-F 0 "C31" H 1570 3770 50  0000 L TNN
+F 0 "C36" H 1570 3770 50  0000 L TNN
 F 1 "0.47u" H 1575 3820 30  0000 L BNN
 	1    1550 3800

Commit message: Changed some values and connected more LCD signals
Parts:
- C42, C43: value 100n -> 0.1u
Changed lines of the file:
@@
-EESchema Schematic File Version 2  date Sun 28 Oct 2012 01:53:13 PM EDT
+EESchema Schematic File Version 2  date Sun 28 Oct 2012 06:31:28 PM EDT
 LIBS:power
 LIBS:device
@@
 P 7950 5150
 F 0 "C43" H 7970 5120 50  0000 L TNN
-F 1 "100n" H 7975 5170 30  0000 L BNN
+F 1 "0.1u" H 7975 5170 30  0000 L BNN
 	1    7950 5150
 	0    -1   -1   0
@@
 P 7000 5800
 F 0 "C42" H 7020 5770 50  0000 L TNN
-F 1 "100n" H 7025 5820 30  0000 L BNN
+F 1 "0.1u" H 7025 5820 30  0000 L BNN
 	1    7000 5800
 	0    -1   -1   0
