File: pcb/audio_in.sch (KiCad schematic (older format))
At the start: 19 parts, among them J5 SJ1-3523N, U11 MCP6409, U12 MCP6241

Commit message: Added comments in the audio section.
Other:
- note added: "Sallen-Key Topology. 2nd order low-pass."
- note added: "Unity Gain buffer to remove the output \nimpedence effect of the audio jack"
Changed lines of the file:
@@
-EESchema Schematic File Version 2  date Mon 14 Jan 2013 05:07:42 PM EST
+EESchema Schematic File Version 2  date Tue 15 Jan 2013 03:28:33 PM EST
 LIBS:power
 LIBS:device
@@
 LIBS:valves
 LIBS:f4_daughter
-LIBS:f4_daughter-cache
 EELAYER 25  0
 EELAYER END
@@
 Sheet 9 9
 Title ""
-Date "14 jan 2013"
+Date "15 jan 2013"
 Rev ""
 Comp ""
@@
 Comment4 ""
 $EndDescr
+Text Notes 3550 2300 0    60   ~ 0
+Sallen-Key Topology. 2nd order low-pass.
+Text Notes 1250 2200 0    60   ~ 0
+Unity Gain buffer to remove the output \nimpedence effect of the audio jack
 Wire Wire Line
 	4400 4300 4350 4300

Commit message: Routing completed, DRC passed
Parts:
- added C53: 0.1u, symbol CAP
Connections:
- wire segments 73 -> 75
Changed lines of the file:
@@
-EESchema Schematic File Version 2  date Thu 17 Jan 2013 04:04:21 PM EST
+EESchema Schematic File Version 2  date Mon 21 Jan 2013 12:51:07 PM EST
 LIBS:power
 LIBS:device
@@
 Sheet 9 9
 Title ""
-Date "17 jan 2013"
+Date "21 jan 2013"
 Rev ""
 Comp ""
@@
 Comment4 ""
 $EndDescr
+Wire Wire Line
+	9100 5350 9100 5250
+Wire Wire Line
+	4400 4300 4350 4300
+Connection ~ 7700 5350
+Wire Wire Line
+	7950 5250 7950 5350
+Wire Wire Line
+	7950 5350 7700 5350
+Connection ~ 7700 4450
+Wire Wire Line
+	8550 4800 8550 4450
+Wire Wire Line
+	8550 4450 7700 4450
+Connection ~ 3000 4100
+Wire Wire Line
+	3000 4100 3000 4450
+Wire Wire Line
+	3000 4450 2200 4450
+Wire Wire Line
+	2200 4450 2200 4200
+Wire Wire Line
+	2200 4200 2300 4200
+Connection ~ 3000 2800
+Wire Wire Line
+	3000 2800 3000 3150
+Wire Wire Line
+	3000 3150 2200 3150
+Wire Wire Line
+	2200 3150 2200 2900
+Wire Wire Line
+	2200 2900 2300 2900
+Wire Wire Line
+	2800 2800 3200 2800
+Wire Wire Line
+	1650 3800 1900 3800
+Wire Wire Line
+	1900 3800 1900 3850
+Wire Wire Line
+	1900 4150 1900 4400
+Wire Wire Line
+	1450 3800 1400 3800
+Wire Wire Line
+	1400 3800 1400 3500
+Wire Wire Line
+	1400 3500 1250 3500
+Wire Wire Line
+	1250 3150 1350 3150
+Wire Wire Line
+	1350 3150 1350 2950
+Wire Wire Line
+	1350 2950 1050 2950
+Wire Wire Line
+	1050 2950 1050 3000
+Wire Wire Line
+	6750 6150 7000 6150
+Connection ~ 6750 6150
+Wire Wire Line
+	7000 6150 7000 5900
+Connection ~ 6750 5450
+Wire Wire Line
+	7000 5700 7000 5450
+Wire Wire Line
+	4100 4450 4100 4550
+Wire Wire Line
+	4100 3250 4100 3150
+Connection ~ 8950 5000
+Wire Wire Line
+	9150 5000 8800 5000
+Wire Wire Line
+	8950 5000 8950 5350
+Wire Wire Line
+	8950 5350 8200 5350
+Wire Wire Line
+	8200 5350 8200 5100
+Wire Wire Line
+	8200 5100 8300 5100
+Wire Wire Line
+	7700 4500 7700 4400
+Connection ~ 5150 4200
+Wire Wire Line
+	5300 4200 4900 4200
+Wire Wire Line
+	5150 4550 5150 3800
+Wire Wire Line
+	5150 4550 4350 4550
+Wire Wire Line
+	4350 4550 4350 4300
+Wire Wire Line
+	7700 5400 7700 5300
+Connection ~ 3550 4100
+Wire Wire Line
+	3600 4100 3450 4100
+Connection ~ 4100 4100
+Wire Wire Line
+	4100 4100 4100 4250
+Wire Wire Line
+	5150 3800 4350 3800
+Wire Wire Line
+	4150 3800 3550 3800
+Wire Wire Line
+	3550 3800 3550 4100
+Connection ~ 7700 4900
+Wire Wire Line
+	8300 4900 7700 4900
+Wire Wire Line
+	7700 5000 7700 4800
+Connection ~ 5150 2900
+Wire Wire Line
+	4350 3250 5150 3250
+Wire Wire Line
+	4350 3250 4350 3000
+Wire Wire Line
+	4350 3000 4450 3000
+Connection ~ 3550 2800
+Wire Wire Line
+	3600 2800 3500 2800
+Connection ~ 4100 2800
+Wire Wire Line
+	4100 2950 4100 2800
+Wire Wire Line
+	4450 2800 3900 2800
+Wire Wire Line
+	5350 2900 4950 2900
+Wire Wire Line
+	5150 3250 5150 2500
+Wire Wire Line
+	5150 2500 4350 2500
+Wire Wire Line
+	4150 2500 3550 2500
+Wire Wire Line
+	3550 2500 3550 2800
+Wire Wire Line
+	6750 6100 6750 6250
+Wire Wire Line
+	6750 5450 6750 5550
+Wire Wire Line
+	1250 3250 1400 3250
+Wire Wire Line
+	1400 3250 1400 2500
+Wire Wire Line
+	1400 2500 1500 2500
+Wire Wire Line
+	1700 2500 1900 2500
+Wire Wire Line
+	1900 2500 1900 2550
+Wire Wire Line
+	1900 2850 1900 3050
+Wire Wire Line
+	2800 4100 3150 4100
+Wire Wire Line
+	2300 2700 2050 2700
+Wire Wire Line
+	2300 4000 2050 4000
+Wire Wire Line
+	8550 5250 8550 5200
+Wire Wire Line
+	7950 5050 7950 4900
+Connection ~ 7950 4900
+Wire Wire Line
+	7000 5450 6700 5450
+Wire Wire Line
+	3900 4100 4400 4100
+Wire Wire Line
+	9100 5050 9100 5000
+Connection ~ 9100 5000
+$Comp
+L GND #PWR056
+U 1 1 50FD74D3
+P 9100 5350
+F 0 "#PWR056" H 9100 5350 30  0001 C CNN
+F 1 "GND" H 9100 5280 30  0001 C CNN
+	1    9100 5350
+	1    0    0    -1
+$EndComp
+$Comp
+L CAP C53
+U 1 1 50FD74C4
+P 9100 5150
+F 0 "C53" H 9120 5120 50  0000 L TNN
+F 1 "0.1u" H 9125 5170 30  0000 L BNN
+	1    9100 5150
+	0    -1   -1   0
+$EndComp
 Text Notes 3550 2300 0    60   ~ 0
 Sallen-Key Topology. 2nd order low-pass.
 Text Notes 1250 2200 0    60   ~ 0
 Unity Gain buffer to remove the output \nimpedence effect of the audio jack
-Wire Wire Line
-	4400 4300 4350 4300
-Connection ~ 7700 5350
-Wire Wire Line
-	7950 5250 7950 5350
-Wire Wire Line
-	7950 5350 7700 5350
-Connection ~ 7700 4450
-Wire Wire Line
-	8550 4800 8550 4450
-Wire Wire Line
-	8550 4450 7700 4450
-Connection ~ 3000 4100
-Wire Wire Line
-	3000 4100 3000 4450
-Wire Wire Line
-	3000 4450 2200 4450
-Wire Wire Line
-	2200 4450 2200 4200
-Wire Wire Line
-	2200 4200 2300 4200
-Connection ~ 3000 2800
-Wire Wire Line
-	3000 2800 3000 3150
-Wire Wire Line
-	3000 3150 2200 3150
-Wire Wire Line
-	2200 3150 2200 2900
-Wire Wire Line
-	2200 2900 2300 2900
-Wire Wire Line
-	2800 2800 3200 2800
-Wire Wire Line
-	1650 3800 1900 3800
-Wire Wire Line
-	1900 3800 1900 3850
-Wire Wire Line
-	1900 4150 1900 4400
-Wire Wire Line
-	1450 3800 1400 3800
-Wire Wire Line
-	1400 3800 1400 3500
-Wire Wire Line
-	1400 3500 1250 3500
-Wire Wire Line
-	1250 3150 1350 3150
-Wire Wire Line
-	1350 3150 1350 2950
-Wire Wire Line
-	1350 2950 1050 2950
-Wire Wire Line
-	1050 2950 1050 3000
-Wire Wire Line
-	6750 6150 7000 6150
-Connection ~ 6750 6150
-Wire Wire Line
-	7000 6150 7000 5900
-Connection ~ 6750 5450
-Wire Wire Line
-	7000 5700 7000 5450
-Wire Wire Line
-	4100 4450 4100 4550
-Wire Wire Line
-	4100 3250 4100 3150
-Connection ~ 8950 5000
-Wire Wire Line
-	9150 5000 8800 5000
-Wire Wire Line
-	8950 5000 8950 5350
-Wire Wire Line
-	8950 5350 8200 5350
-Wire Wire Line
-	8200 5350 8200 5100
-Wire Wire Line
-	8200 5100 8300 5100
-Wire Wire Line
-	7700 4500 7700 4400
-Connection ~ 5150 4200
-Wire Wire Line
-	5300 4200 4900 4200
-Wire Wire Line
-	5150 4550 5150 3800
-Wire Wire Line
-	5150 4550 4350 4550
-Wire Wire Line
-	4350 4550 4350 4300
-Wire Wire Line
-	7700 5400 7700 5300
-Connection ~ 3550 4100
-Wire Wire Line
-	3600 4100 3450 4100
-Connection ~ 4100 4100
-Wire Wire Line
-	4100 4100 4100 4250
-Wire Wire Line
-	5150 3800 4350 3800
-Wire Wire Line
-	4150 3800 3550 3800
-Wire Wire Line
-	3550 3800 3550 4100
-Connection ~ 7700 4900
-Wire Wire Line
-	8300 4900 7700 4900
-Wire Wire Line
-	7700 5000 7700 4800
-Connection ~ 5150 2900
-Wire Wire Line
-	4350 3250 5150 3250
-Wire Wire Line
-	4350 3250 4350 3000
-Wire Wire Line
-	4350 3000 4450 3000
-Connection ~ 3550 2800
-Wire Wire Line
-	3600 2800 3500 2800
-Connection ~ 4100 2800
-Wire Wire Line
-	4100 2950 4100 2800
-Wire Wire Line
-	4450 2800 3900 2800
-Wire Wire Line
-	5350 2900 4950 2900
-Wire Wire Line
-	5150 3250 5150 2500
-Wire Wire Line
-	5150 2500 4350 2500
-Wire Wire Line
-	4150 2500 3550 2500
-Wire Wire Line
-	3550 2500 3550 2800
-Wire Wire Line
-	6750 6100 6750 6250
-Wire Wire Line
-	6750 5450 6750 5550
-Wire Wire Line
-	1250 3250 1400 3250
-Wire Wire Line
-	1400 3250 1400 2500
-Wire Wire Line
-	1400 2500 1500 2500
-Wire Wire Line
-	1700 2500 1900 2500
-Wire Wire Line
-	1900 2500 1900 2550
-Wire Wire Line
-	1900 2850 1900 3050
-Wire Wire Line
-	2800 4100 3150 4100
-Wire Wire Line
-	2300 2700 2050 2700
-Wire Wire Line
-	2300 4000 2050 4000
-Wire Wire Line
-	8550 5250 8550 5200
-Wire Wire Line
-	7950 5050 7950 4900
-Connection ~ 7950 4900
-Wire Wire Line
-	7000 5450 6700 5450
-Wire Wire Line
-	3900 4100 4400 4100
 $Comp
 L CAP C43
@@
 $EndComp
 $Comp
-L GND #PWR056
+L GND #PWR057
 U 1 1 504649EC
 P 8550 5250
-F 0 "#PWR056" H 8550 5250 30  0001 C CNN
+F 0 "#PWR057" H 8550 5250 30  0001 C CNN
 F 1 "GND" H 8550 5180 30  0001 C CNN
 	1    8550 5250
@@
 VGND
 $Comp
-L GND #PWR057
+L GND #PWR058
 U 1 1 50118BD6
 P 1050 3000
-F 0 "#PWR057" H 1050 3000 30  0001 C CNN
+F 0 "#PWR058" H 1050 3000 30  0001 C CNN
 F 1 "GND" H 1050 2930 30  0001 C CNN
 	1    1050 3000
@@
 Vreg
 $Comp
-L GND #PWR058
+L GND #PWR059
 U 1 1 5010D90D
 P 6750 6250
-F 0 "#PWR058" H 6750 6250 30  0001 C CNN
+F 0 "#PWR059" H 6750 6250 30  0001 C CNN
 F 1 "GND" H 6750 6180 30  0001 C CNN
 	1    6750 6250
@@
 Vreg
 $Comp
-L GND #PWR059
+L GND #PWR060
 U 1 1 5010DA28
 P 7700 5400
-F 0 "#PWR059" H 7700 5400 30  0001 C CNN
+F 0 "#PWR060" H 7700 5400 30  0001 C CNN
 F 1 "GND" H 7700 5330 30  0001 C CNN
 	1    7700 5400

Commit message: Added comment in audio sheet explaining VGND.
Other:
- note added: "VGND Node production so that it is at Vreg/2.\nThe rails go from GND to Vreg."
Changed lines of the file:
@@
-EESchema Schematic File Version 2  date Mon 21 Jan 2013 12:51:07 PM EST
+EESchema Schematic File Version 2  date Mon 21 Jan 2013 04:13:24 PM EST
 LIBS:power
 LIBS:device
@@
 Comment4 ""
 $EndDescr
+Text Notes 7450 4000 0    60   ~ 0
+VGND Node production so that it is at Vreg/2.\nThe rails go from GND to Vreg.
 Wire Wire Line
 	9100 5350 9100 5250
