File: pcb/rf.sch (KiCad schematic (older format))
At the start: 29 parts, among them T1 TP, U3 STM32W108C8, U4 SE2432L, U9 SN74LVC1G125

Commit message: Added crystal, 2nd antenna, and SWD for STM32W
Parts:
- added C? (x2): CAP, symbol CAP
- added J3: 73391-0070, symbol COAX
- added J4: CONN_6, symbol CONN_6
- added R6: 180k, symbol RES
- added X?: XTAL, symbol XTAL
Connections:
- net labels added: PB5, SWCLK, SWDIO, SWO
- net labels removed: RF_RESET
- wire segments 140 -> 179
Other:
- note added: "DO NOT POPULATE"
- note added: "SWD Header"
- moved on the sheet: C18, C19

Commit message: Added battery level detection. This changed the annotation in other files as well.
Parts:
- gave numbers to parts that had none: 2
Changed lines of the file:
@@
-EESchema Schematic File Version 2  date Tue 09 Oct 2012 06:48:49 PM EDT
+EESchema Schematic File Version 2  date 10/10/2012 1:41:54 PM
 LIBS:power
 LIBS:device
@@
 Sheet 4 7
 Title ""
-Date "9 oct 2012"
+Date "10 oct 2012"
 Rev ""
 Comp ""
@@
 Connection ~ 6250 2700
 $Comp
-L GND #PWR?
+L GND #PWR21
 U 1 1 5074807E
 P 6400 2300
-F 0 "#PWR?" H 6400 2300 30  0001 C CNN
+F 0 "#PWR21" H 6400 2300 30  0001 C CNN
 F 1 "GND" H 6400 2230 30  0001 C CNN
 	1    6400 2300
@@
 $EndComp
 $Comp
-L CAP C?
+L CAP C43
 U 1 1 50748076
 P 6550 2450
-F 0 "C?" H 6570 2420 50  0000 L TNN
+F 0 "C43" H 6570 2420 50  0000 L TNN
 F 1 "CAP" H 6575 2470 30  0000 L BNN
 	1    6550 2450
@@
 $EndComp
 $Comp
-L CAP C?
+L CAP C42
 U 1 1 50748074
 P 6250 2450
-F 0 "C?" H 6270 2420 50  0000 L TNN
+F 0 "C42" H 6270 2420 50  0000 L TNN
 F 1 "CAP" H 6275 2470 30  0000 L BNN
 	1    6250 2450
@@
 RESET
 $Comp
-L GND #PWR25
+L GND #PWR27
 U 1 1 5074771B
 P 8950 3850
-F 0 "#PWR25" H 8950 3850 30  0001 C CNN
+F 0 "#PWR27" H 8950 3850 30  0001 C CNN
 F 1 "GND" H 8950 3780 30  0001 C CNN
 	1    8950 3850
@@
 $EndComp
 $Comp
-L GND #PWR12
+L GND #PWR13
 U 1 1 507475AD
 P 2350 3900
-F 0 "#PWR12" H 2350 3900 30  0001 C CNN
+F 0 "#PWR13" H 2350 3900 30  0001 C CNN
 F 1 "GND" H 2350 3830 30  0001 C CNN
 	1    2350 3900
@@
 $EndComp
 $Comp
-L GND #PWR14
+L GND #PWR15
 U 1 1 507472EA
 P 3250 4450
-F 0 "#PWR14" H 3250 4450 30  0001 C CNN
+F 0 "#PWR15" H 3250 4450 30  0001 C CNN
 F 1 "GND" H 3250 4380 30  0001 C CNN
 	1    3250 4450
@@
 PB5
 $Comp
-L GND #PWR20
+L GND #PWR22
 U 1 1 50196BA7
 P 7300 6500
-F 0 "#PWR20" H 7300 6500 30  0001 C CNN
+F 0 "#PWR22" H 7300 6500 30  0001 C CNN
 F 1 "GND" H 7300 6430 30  0001 C CNN
 	1    7300 6500
@@
 PC5
 $Comp
-L GND #PWR24
+L GND #PWR26
 U 1 1 500DD937
 P 8250 4650
-F 0 "#PWR24" H 8250 4650 30  0001 C CNN
+F 0 "#PWR26" H 8250 4650 30  0001 C CNN
 F 1 "GND" H 8250 4580 30  0001 C CNN
 	1    8250 4650
@@
 $EndComp
 $Comp
-L GND #PWR23
+L GND #PWR25
 U 1 1 500DD883
 P 8100 3050
-F 0 "#PWR23" H 8100 3050 30  0001 C CNN
+F 0 "#PWR25" H 8100 3050 30  0001 C CNN
 F 1 "GND" H 8100 2980 30  0001 C CNN
 	1    8100 3050
@@
 1V2
 $Comp
-L GND #PWR18
+L GND #PWR19
 U 1 1 500DD7C0
 P 5800 2900
-F 0 "#PWR18" H 5800 2900 30  0001 C CNN
+F 0 "#PWR19" H 5800 2900 30  0001 C CNN
 F 1 "GND" H 5800 2830 30  0001 C CNN
 	1    5800 2900
@@
 $EndComp
 $Comp
-L GND #PWR21
+L GND #PWR23
 U 1 1 500DD6F0
 P 7550 5650
-F 0 "#PWR21" H 7550 5650 30  0001 C CNN
+F 0 "#PWR23" H 7550 5650 30  0001 C CNN
 F 1 "GND" H 7550 5580 30  0001 C CNN
 	1    7550 5650
@@
 Vreg
 $Comp
-L GND #PWR16
+L GND #PWR17
 U 1 1 500DD2FF
 P 5000 3650
-F 0 "#PWR16" H 5000 3650 30  0001 C CNN
+F 0 "#PWR17" H 5000 3650 30  0001 C CNN
 F 1 "GND" H 5000 3580 30  0001 C CNN
 	1    5000 3650
@@
 $EndComp
 $Comp
-L GND #PWR19
+L GND #PWR20
 U 1 1 500DD1EA
 P 6000 5850
-F 0 "#PWR19" H 6000 5850 30  0001 C CNN
+F 0 "#PWR20" H 6000 5850 30  0001 C CNN
 F 1 "GND" H 6000 5780 30  0001 C CNN
 	1    6000 5850
@@
 $EndComp
 $Comp
-L GND #PWR17
+L GND #PWR18
 U 1 1 500DCCCC
 P 5550 5050
-F 0 "#PWR17" H 5550 5050 30  0001 C CNN
+F 0 "#PWR18" H 5550 5050 30  0001 C CNN
 F 1 "GND" H 5550 4980 30  0001 C CNN
 	1    5550 5050
@@
 1V8
 $Comp
-L GND #PWR13
+L GND #PWR14
 U 1 1 500DCAB4
 P 3050 4500
-F 0 "#PWR13" H 3050 4500 30  0001 C CNN
+F 0 "#PWR14" H 3050 4500 30  0001 C CNN
 F 1 "GND" H 3050 4430 30  0001 C CNN
 	1    3050 4500
@@
 $EndComp
 $Comp
-L GND #PWR11
+L GND #PWR12
 U 1 1 500DCAB1
 P 2200 4500
-F 0 "#PWR11" H 2200 4500 30  0001 C CNN
+F 0 "#PWR12" H 2200 4500 30  0001 C CNN
 F 1 "GND" H 2200 4430 30  0001 C CNN
 	1    2200 4500
@@
 $EndComp
 $Comp
-L GND #PWR15
+L GND #PWR16
 U 1 1 500DCAA7
 P 3650 3950
-F 0 "#PWR15" H 3650 3950 30  0001 C CNN
+F 0 "#PWR16" H 3650 3950 30  0001 C CNN
 F 1 "GND" H 3650 3880 30  0001 C CNN
 	1    3650 3950
@@
 $EndComp
 $Comp
-L GND #PWR10
+L GND #PWR11
 U 1 1 500DCA40
 P 1800 4200
-F 0 "#PWR10" H 1800 4200 30  0001 C CNN
+F 0 "#PWR11" H 1800 4200 30  0001 C CNN
 F 1 "GND" H 1800 4130 30  0001 C CNN
 	1    1800 4200
@@
 $EndComp
 $Comp
-L GND #PWR22
+L GND #PWR24
 U 1 1 500DCA3C
 P 8050 4950
-F 0 "#PWR22" H 8050 4950 30  0001 C CNN
+F 0 "#PWR24" H 8050 4950 30  0001 C CNN
 F 1 "GND" H 8050 4880 30  0001 C CNN
 	1    8050 4950

Commit message: Reannoted everything so that there isn't any duplicates. Also added connection to the rf reset line.
Parts:
- renumbered C15 to C10, C18 to C11, C16 to C12, C19 to C13, C17 to C14, C42 to C15, C43 to C16, C20 to C17, C21 to C18, C22 to C19, C23 to C20, C24 to C21, C25 to C22, C8 to C3, C9 to C4, C10 to C5, C11 to C6, C12 to C7, C13 to C8, C14 to C9, J3 to J2, J4 to J3, L4 to L1, R3 to R10, R4 to R11, R5 to R12, R6 to R13, R1 to R8, R2 to R9, U3 to U5, U9 to U6

Commit message: A few things: Remapped all interrupts and identified unusable pins on board Added all required connections for LCD and company Added pull-down resistor on STM32W Renamed some internal signals on RF for consistency
Parts:
- added R?: 180k, symbol RES
Connections:
- net labels removed: SPI1_CLK, SPI1_MISO, SPI1_MOSI
- wire segments 179 -> 182
Other:
- note added: "RF SWD Header"
- note removed: "SWD Header"
- moved on the sheet: R13

Commit message: A few more things: Added low-voltage battery detection to disable regulators Fixed XTAL symbol Annotated new components from yesterday
Parts:
- gave numbers to parts that had none: 2
Changed lines of the file:
@@
-EESchema Schematic File Version 2  date Sat 27 Oct 2012 09:22:30 PM EDT
+EESchema Schematic File Version 2  date Sun 28 Oct 2012 01:53:13 PM EDT
 LIBS:power
 LIBS:device
@@
 $Descr A4 11700 8267
 encoding utf-8
-Sheet 4 7
+Sheet 5 7
 Title ""
 Date "28 oct 2012"
@@
 $EndDescr
 Wire Wire Line
+	6500 2700 6550 2700
+Wire Wire Line
 	5750 4600 5950 4600
 Connection ~ 9750 3100
@@
 	9750 3300 9750 3100
 Connection ~ 6250 2700
-Wire Wire Line
-	6300 2700 6250 2700
 Wire Wire Line
 	6550 2800 6450 2800
@@
 Wire Wire Line
 	6250 2800 6250 2550
-Wire Wire Line
-	6500 2700 6550 2700
 Connection ~ 6550 2700
 Wire Wire Line
@@
 Wire Wire Line
 	9250 3300 9350 3300
-$Comp
-L GND #PWR?
+Wire Wire Line
+	6300 2700 6250 2700
+$Comp
+L GND #PWR31
 U 1 1 508C84BE
 P 9250 3400
-F 0 "#PWR?" H 9250 3400 30  0001 C CNN
+F 0 "#PWR31" H 9250 3400 30  0001 C CNN
 F 1 "GND" H 9250 3330 30  0001 C CNN
 	1    9250 3400
@@
 $EndComp
 $Comp
-L RES R?
+L RES R34
 U 1 1 508C84A1
 P 9500 3300
-F 0 "R?" H 9570 3265 50  0000 L TNN
+F 0 "R34" H 9570 3265 50  0000 L TNN
 F 1 "180k" H 9500 3355 30  0000 C BNN
 	1    9500 3300
@@
 $EndComp
 $Comp
-L GND #PWR23
+L GND #PWR24
 U 1 1 5074807E
 P 6400 2300
-F 0 "#PWR23" H 6400 2300 30  0001 C CNN
+F 0 "#PWR24" H 6400 2300 30  0001 C CNN
 F 1 "GND" H 6400 2230 30  0001 C CNN
 	1    6400 2300
@@
 $EndComp
 $Comp
-L XTAL X?
+L XTAL X1
 U 1 1 50748066
 P 6400 2700
-F 0 "X?" H 6400 2640 40  0000 C TNN
+F 0 "X1" H 6400 2640 40  0000 C TNN
 F 1 "XTAL" H 6400 2760 40  0000 C BNN
 	1    6400 2700
@@
 RESET
 $Comp
-L GND #PWR29
+L GND #PWR30
 U 1 1 5074771B
 P 8950 3850
-F 0 "#PWR29" H 8950 3850 30  0001 C CNN
+F 0 "#PWR30" H 8950 3850 30  0001 C CNN
 F 1 "GND" H 8950 3780 30  0001 C CNN
 	1    8950 3850
@@
 $EndComp
 $Comp
-L GND #PWR15
+L GND #PWR16
 U 1 1 507475AD
 P 2350 3900
-F 0 "#PWR15" H 2350 3900 30  0001 C CNN
+F 0 "#PWR16" H 2350 3900 30  0001 C CNN
 F 1 "GND" H 2350 3830 30  0001 C CNN
 	1    2350 3900
@@
 $EndComp
 $Comp
-L GND #PWR17
+L GND #PWR18
 U 1 1 507472EA
 P 3250 4450
-F 0 "#PWR17" H 3250 4450 30  0001 C CNN
+F 0 "#PWR18" H 3250 4450 30  0001 C CNN
 F 1 "GND" H 3250 4380 30  0001 C CNN
 	1    3250 4450
@@
 PB5
 $Comp
-L GND #PWR24
+L GND #PWR25
 U 1 1 50196BA7
 P 7300 6500
-F 0 "#PWR24" H 7300 6500 30  0001 C CNN
+F 0 "#PWR25" H 7300 6500 30  0001 C CNN
 F 1 "GND" H 7300 6430 30  0001 C CNN
 	1    7300 6500
@@
 PC5
 $Comp
-L GND #PWR28
+L GND #PWR29
 U 1 1 500DD937
 P 8250 4650
-F 0 "#PWR28" H 8250 4650 30  0001 C CNN
+F 0 "#PWR29" H 8250 4650 30  0001 C CNN
 F 1 "GND" H 8250 4580 30  0001 C CNN
 	1    8250 4650
@@
 $EndComp
 $Comp
-L GND #PWR27
+L GND #PWR28
 U 1 1 500DD883
 P 8100 3050
-F 0 "#PWR27" H 8100 3050 30  0001 C CNN
+F 0 "#PWR28" H 8100 3050 30  0001 C CNN
 F 1 "GND" H 8100 2980 30  0001 C CNN
 	1    8100 3050
@@
 1V2
 $Comp
-L GND #PWR21
+L GND #PWR22
 U 1 1 500DD7C0
 P 5800 2900
-F 0 "#PWR21" H 5800 2900 30  0001 C CNN
+F 0 "#PWR22" H 5800 2900 30  0001 C CNN
 F 1 "GND" H 5800 2830 30  0001 C CNN
 	1    5800 2900
@@
 $EndComp
 $Comp
-L GND #PWR25
+L GND #PWR26
 U 1 1 500DD6F0
 P 7550 5650
-F 0 "#PWR25" H 7550 5650 30  0001 C CNN
+F 0 "#PWR26" H 7550 5650 30  0001 C CNN
 F 1 "GND" H 7550 5580 30  0001 C CNN
 	1    7550 5650
@@
 Vreg
 $Comp
-L GND #PWR19
+L GND #PWR20
 U 1 1 500DD2FF
 P 5000 3650
-F 0 "#PWR19" H 5000 3650 30  0001 C CNN
+F 0 "#PWR20" H 5000 3650 30  0001 C CNN
 F 1 "GND" H 5000 3580 30  0001 C CNN
 	1    5000 3650
@@
 $EndComp
 $Comp
-L GND #PWR22
+L GND #PWR23
 U 1 1 500DD1EA
 P 6000 5850
-F 0 "#PWR22" H 6000 5850 30  0001 C CNN
+F 0 "#PWR23" H 6000 5850 30  0001 C CNN
 F 1 "GND" H 6000 5780 30  0001 C CNN
 	1    6000 5850
@@
 $EndComp
 $Comp
-L GND #PWR20
+L GND #PWR21
 U 1 1 500DCCCC
 P 5550 5050
-F 0 "#PWR20" H 5550 5050 30  0001 C CNN
+F 0 "#PWR21" H 5550 5050 30  0001 C CNN
 F 1 "GND" H 5550 4980 30  0001 C CNN
 	1    5550 5050
@@
 1V8
 $Comp
-L GND #PWR16
+L GND #PWR17
 U 1 1 500DCAB4
 P 3050 4500
-F 0 "#PWR16" H 3050 4500 30  0001 C CNN
+F 0 "#PWR17" H 3050 4500 30  0001 C CNN
 F 1 "GND" H 3050 4430 30  0001 C CNN
 	1    3050 4500
@@
 $EndComp
 $Comp
-L GND #PWR14
+L GND #PWR15
 U 1 1 500DCAB1
 P 2200 4500
-F 0 "#PWR14" H 2200 4500 30  0001 C CNN
+F 0 "#PWR15" H 2200 4500 30  0001 C CNN
 F 1 "GND" H 2200 4430 30  0001 C CNN
 	1    2200 4500
@@
 $EndComp
 $Comp
-L GND #PWR18
+L GND #PWR19
 U 1 1 500DCAA7
 P 3650 3950
-F 0 "#PWR18" H 3650 3950 30  0001 C CNN
+F 0 "#PWR19" H 3650 3950 30  0001 C CNN
 F 1 "GND" H 3650 3880 30  0001 C CNN
 	1    3650 3950
@@
 $EndComp
 $Comp
-L GND #PWR13
+L GND #PWR14
 U 1 1 500DCA40
 P 1800 4200
-F 0 "#PWR13" H 1800 4200 30  0001 C CNN
+F 0 "#PWR14" H 1800 4200 30  0001 C CNN
 F 1 "GND" H 1800 4130 30  0001 C CNN
 	1    1800 4200
@@
 $EndComp
 $Comp
-L GND #PWR26
+L GND #PWR27
 U 1 1 500DCA3C
 P 8050 4950
-F 0 "#PWR26" H 8050 4950 30  0001 C CNN
+F 0 "#PWR27" H 8050 4950 30  0001 C CNN
 F 1 "GND" H 8050 4880 30  0001 C CNN
 	1    8050 4950

Commit message: Changed some values and connected more LCD signals
Parts:
- C11: value 1n -> 1000p
- C12, C13, C19: value 10n -> 0.01u
- C17, C20, C21, C22, C6, C8: value 100n -> 0.1u
- C18: value 100n -> 01.u
Changed lines of the file:
@@
-EESchema Schematic File Version 2  date Sun 28 Oct 2012 01:53:13 PM EDT
+EESchema Schematic File Version 2  date Sun 28 Oct 2012 06:31:28 PM EDT
 LIBS:power
 LIBS:device
@@
 P 8250 4450
 F 0 "C22" H 8270 4420 50  0000 L TNN
-F 1 "100n" H 8275 4470 30  0000 L BNN
+F 1 "0.1u" H 8275 4470 30  0000 L BNN
 	1    8250 4450
 	0    1    1    0
@@
 P 7900 2950
 F 0 "C21" H 7920 2920 50  0000 L TNN
-F 1 "100n" H 7925 2970 30  0000 L BNN
+F 1 "0.1u" H 7925 2970 30  0000 L BNN
 	1    7900 2950
 	-1   0    0    1
@@
 P 5900 2700
 F 0 "C13" H 5920 2670 50  0000 L TNN
-F 1 "10n" H 5925 2720 30  0000 L BNN
+F 1 "0.01u" H 5925 2720 30  0000 L BNN
 	1    5900 2700
 	0    -1   -1   0
@@
 P 5700 2700
 F 0 "C11" H 5720 2670 50  0000 L TNN
-F 1 "1n" H 5725 2720 30  0000 L BNN
+F 1 "1000p" H 5725 2720 30  0000 L BNN
 	1    5700 2700
 	0    -1   -1   0
@@
 P 6650 5650
 F 0 "C17" H 6475 5725 50  0000 L TNN
-F 1 "100n" H 6675 5670 30  0000 L BNN
+F 1 "0.1u" H 6675 5670 30  0000 L BNN
 	1    6650 5650
 	0    -1   -1   0
@@
 P 6900 5500
 F 0 "C19" H 6920 5470 50  0000 L TNN
-F 1 "10n" H 6925 5520 30  0000 L BNN
+F 1 "0.01u" H 6925 5520 30  0000 L BNN
 	1    6900 5500
 	0    -1   -1   0
@@
 P 6750 5500
 F 0 "C18" H 6575 5475 50  0000 L TNN
-F 1 "100n" H 6775 5520 30  0000 L BNN
+F 1 "01.u" H 6775 5520 30  0000 L BNN
 	1    6750 5500
 	0    -1   -1   0
@@
 P 7550 5450
 F 0 "C20" H 7570 5420 50  0000 L TNN
-F 1 "100n" H 7575 5470 30  0000 L BNN
+F 1 "0.1u" H 7575 5470 30  0000 L BNN
 	1    7550 5450
 	0    -1   -1   0
@@
 P 5850 5600
 F 0 "C12" H 5870 5570 50  0000 L TNN
-F 1 "10n" H 5875 5620 30  0000 L BNN
+F 1 "0.01u" H 5875 5620 30  0000 L BNN
 	1    5850 5600
 	0    -1   -1   0
@@
 P 4150 5100
 F 0 "C8" H 4170 5070 50  0000 L TNN
-F 1 "100n" H 4175 5120 30  0000 L BNN
+F 1 "0.1u" H 4175 5120 30  0000 L BNN
 	1    4150 5100
 	0    -1   -1   0
@@
 P 3700 5100
 F 0 "C6" H 3720 5070 50  0000 L TNN
-F 1 "100n" H 3725 5120 30  0000 L BNN
+F 1 "0.1u" H 3725 5120 30  0000 L BNN
 	1    3700 5100
 	0    -1   -1   0
