File: pcb/rf.sch (KiCad schematic (older format))
At the start: 36 parts, among them J2 73391-0070, J3 CONN_6, T1 TP, U4 SE2432L, U5 STM32W108C8, U6 SN74LVC1G125, X1 XTAL

Commit message: Replaced the old antenna symbol with the new one
Parts:
- removed J2: 73391-0070, symbol COAX
- added J?: 73391-0070, symbol 73391-0070
Connections:
- wire segments 182 -> 185

Commit message: Added the annotation for the antenna
Parts:
- gave numbers to parts that had none: 1
Changed lines of the file:
@@
-EESchema Schematic File Version 2  date 1/8/2013 3:03:22 PM
+EESchema Schematic File Version 2  date 1/8/2013 3:07:46 PM
 LIBS:power
 LIBS:device
@@
 $EndComp
 $Comp
-L 73391-0070 J?
+L 73391-0070 J2
 U 1 1 50EC7B2B
 P 2600 3650
-F 0 "J?" H 3000 3400 60  0000 C CNN
+F 0 "J2" H 3000 3400 60  0000 C CNN
 F 1 "73391-0070" H 2950 3800 60  0000 C CNN
 	1    2600 3650

Commit message: Cleaned up antenna symbols and more footprint associations
Parts:
- removed J2: 73391-0070, symbol 73391-0070
- added E2: COAX, symbol COAX
- C18: value 01.u -> 0.1u
Connections:
- wire segments 185 -> 183

Commit message: Starting layout.
Connections:
- wire segments 183 -> 182
Changed lines of the file:
@@
-EESchema Schematic File Version 2  date Wed 09 Jan 2013 04:33:42 PM EST
+EESchema Schematic File Version 2  date 1/9/2013 5:22:51 PM
 LIBS:power
 LIBS:device
@@
 Comment4 ""
 $EndDescr
+$Comp
+L SE2432L U4
+U 1 1 50EDED7A
+P 4450 4100
+F 0 "U4" H 4750 3550 60  0000 C CNN
+F 1 "SE2432L" H 4900 4650 60  0000 C CNN
+	1    4450 4100
+	1    0    0    -1
+$EndComp
 Wire Wire Line
 	6750 5850 6750 5600
@@
 Wire Wire Line
 	3750 4000 3950 4000
-Wire Wire Line
-	3850 3650 3650 3650
 Connection ~ 3650 3900
 Wire Wire Line
@@
 Wire Wire Line
 	3650 3450 3650 3950
-Connection ~ 3650 3650
 Connection ~ 4250 3450
 Wire Wire Line
@@
 	2350 3650 2400 3650
 $Comp
-L GND #PWR?
+L GND #PWR016
 U 1 1 50EDE224
 P 6750 5850
-F 0 "#PWR?" H 6750 5850 30  0001 C CNN
+F 0 "#PWR016" H 6750 5850 30  0001 C CNN
 F 1 "GND" H 6750 5780 30  0001 C CNN
 	1    6750 5850
@@
 $EndComp
 $Comp
-L GND #PWR016
+L GND #PWR017
 U 1 1 50EDDFB8
 P 2350 3750
-F 0 "#PWR016" H 2350 3750 30  0001 C CNN
+F 0 "#PWR017" H 2350 3750 30  0001 C CNN
 F 1 "GND" H 2350 3680 30  0001 C CNN
 	1    2350 3750
@@
 $EndComp
 $Comp
-L GND #PWR017
+L GND #PWR018
 U 1 1 508C84BE
 P 9250 3400
-F 0 "#PWR017" H 9250 3400 30  0001 C CNN
+F 0 "#PWR018" H 9250 3400 30  0001 C CNN
 F 1 "GND" H 9250 3330 30  0001 C CNN
 	1    9250 3400
@@
 $EndComp
 $Comp
-L GND #PWR018
+L GND #PWR019
 U 1 1 5074807E
 P 6400 2300
-F 0 "#PWR018" H 6400 2300 30  0001 C CNN
+F 0 "#PWR019" H 6400 2300 30  0001 C CNN
 F 1 "GND" H 6400 2230 30  0001 C CNN
 	1    6400 2300
@@
 RESET
 $Comp
-L GND #PWR019
+L GND #PWR020
 U 1 1 5074771B
 P 8950 3850
-F 0 "#PWR019" H 8950 3850 30  0001 C CNN
+F 0 "#PWR020" H 8950 3850 30  0001 C CNN
 F 1 "GND" H 8950 3780 30  0001 C CNN
 	1    8950 3850
@@
 $EndComp
 $Comp
-L GND #PWR020
+L GND #PWR021
 U 1 1 507472EA
 P 3250 4450
-F 0 "#PWR020" H 3250 4450 30  0001 C CNN
+F 0 "#PWR021" H 3250 4450 30  0001 C CNN
 F 1 "GND" H 3250 4380 30  0001 C CNN
 	1    3250 4450
@@
 PB5
 $Comp
-L GND #PWR021
+L GND #PWR022
 U 1 1 50196BA7
 P 7300 6500
-F 0 "#PWR021" H 7300 6500 30  0001 C CNN
+F 0 "#PWR022" H 7300 6500 30  0001 C CNN
 F 1 "GND" H 7300 6430 30  0001 C CNN
 	1    7300 6500
@@
 PC5
 $Comp
-L GND #PWR022
+L GND #PWR023
 U 1 1 500DD937
 P 8250 4650
-F 0 "#PWR022" H 8250 4650 30  0001 C CNN
+F 0 "#PWR023" H 8250 4650 30  0001 C CNN
 F 1 "GND" H 8250 4580 30  0001 C CNN
 	1    8250 4650
@@
 $EndComp
 $Comp
-L GND #PWR023
+L GND #PWR024
 U 1 1 500DD883
 P 8100 3050
-F 0 "#PWR023" H 8100 3050 30  0001 C CNN
+F 0 "#PWR024" H 8100 3050 30  0001 C CNN
 F 1 "GND" H 8100 2980 30  0001 C CNN
 	1    8100 3050
@@
 1V2
 $Comp
-L GND #PWR024
+L GND #PWR025
 U 1 1 500DD7C0
 P 5800 2900
-F 0 "#PWR024" H 5800 2900 30  0001 C CNN
+F 0 "#PWR025" H 5800 2900 30  0001 C CNN
 F 1 "GND" H 5800 2830 30  0001 C CNN
 	1    5800 2900
@@
 $EndComp
 $Comp
-L GND #PWR025
+L GND #PWR026
 U 1 1 500DD6F0
 P 7550 5650
-F 0 "#PWR025" H 7550 5650 30  0001 C CNN
+F 0 "#PWR026" H 7550 5650 30  0001 C CNN
 F 1 "GND" H 7550 5580 30  0001 C CNN
 	1    7550 5650
@@
 Vreg
 $Comp
-L GND #PWR026
+L GND #PWR027
 U 1 1 500DD2FF
 P 5000 3650
-F 0 "#PWR026" H 5000 3650 30  0001 C CNN
+F 0 "#PWR027" H 5000 3650 30  0001 C CNN
 F 1 "GND" H 5000 3580 30  0001 C CNN
 	1    5000 3650
@@
 $EndComp
 $Comp
-L GND #PWR027
+L GND #PWR028
 U 1 1 500DD1EA
 P 6000 5850
-F 0 "#PWR027" H 6000 5850 30  0001 C CNN
+F 0 "#PWR028" H 6000 5850 30  0001 C CNN
 F 1 "GND" H 6000 5780 30  0001 C CNN
 	1    6000 5850
@@
 $EndComp
 $Comp
-L GND #PWR028
+L GND #PWR029
 U 1 1 500DCCCC
 P 5550 5050
-F 0 "#PWR028" H 5550 5050 30  0001 C CNN
+F 0 "#PWR029" H 5550 5050 30  0001 C CNN
 F 1 "GND" H 5550 4980 30  0001 C CNN
 	1    5550 5050
@@
 1V8
 $Comp
-L GND #PWR029
+L GND #PWR030
 U 1 1 500DCAB4
 P 3050 4500
-F 0 "#PWR029" H 3050 4500 30  0001 C CNN
+F 0 "#PWR030" H 3050 4500 30  0001 C CNN
 F 1 "GND" H 3050 4430 30  0001 C CNN
 	1    3050 4500
@@
 $EndComp
 $Comp
-L GND #PWR030
+L GND #PWR031
 U 1 1 500DCAB1
 P 2200 4500
-F 0 "#PWR030" H 2200 4500 30  0001 C CNN
+F 0 "#PWR031" H 2200 4500 30  0001 C CNN
 F 1 "GND" H 2200 4430 30  0001 C CNN
 	1    2200 4500
@@
 $EndComp
 $Comp
-L GND #PWR031
+L GND #PWR032
 U 1 1 500DCAA7
 P 3650 3950
-F 0 "#PWR031" H 3650 3950 30  0001 C CNN
+F 0 "#PWR032" H 3650 3950 30  0001 C CNN
 F 1 "GND" H 3650 3880 30  0001 C CNN
 	1    3650 3950
@@
 $EndComp
 $Comp
-L GND #PWR032
+L GND #PWR033
 U 1 1 500DCA3C
 P 8050 4950
-F 0 "#PWR032" H 8050 4950 30  0001 C CNN
+F 0 "#PWR033" H 8050 4950 30  0001 C CNN
 F 1 "GND" H 8050 4880 30  0001 C CNN
 	1    8050 4950
@@
 $EndComp
 $Comp
-L SE2432L U4
-U 1 1 500DCA0F
-P 4450 4100
-F 0 "U4" H 4750 3550 60  0000 C CNN
-F 1 "SE2432L" H 4900 4650 60  0000 C CNN
-	1    4450 4100
-	-1   0    0    1
-$EndComp
-$Comp
