File: pcb/cpld.sch (KiCad schematic (older format))
At the start: 1 part

Commit message: Restored CPLD sheet.
Parts:
- removed U?: XC2C64A-XQFG48, symbol XC2C64A-XQFG48
- added P?: CONN_5, symbol CONN_5
- added S? (x4): EVQ-Q2S03W, symbol EVQ-Q2S03W
- added U?: XC2C64A-XQFG48, symbol XC2C64A-XQFG48
Connections:
- net labels added: EXTI0, EXTI1, EXTI11, EXTI12, EXTI13, EXTI15, EXTI2, EXTI3, EXTI4, EXTI5, EXTI6, EXTI7, EXTI8, FSMC_A16, FSMC_NEx, FSMC_NWE, INT1_ACC, INT1_GYR, INT2_ACC, INT2_GYR, INT2_GYR/DRDY, JTCK, JTDI, JTDO, JTMS, POW_HPWR, POW_MODE, POW_NXT, RF_IRQ, RS, S1, S2, S3, S4, SPI_MISO, SPI_MOSI, SPI_NCS, SPI_SCK, TOUCH_IRQ, VCC_JTAG, nCS, nRD, nWR
- net labels removed: 1.10(GTS0), 1.3, 1.9(GTS1), V1.8
- wire segments 12 -> 113
Other:
- note added: "Daughter Board I/O"
- note added: "Discovery Board I/O"
- note added: "JTAG Header"
- note added: "Suggested Interrupt Setup:\nIndependent Vectors:\n EXTI0: LIS302_INT1\n EXTI1: LIS302_INT2\n EXTI2: SPI_IRQ_RF\n EXTI3: SPI_IRQ_TOUCH\n EXTI4:\n\nEXTI9_5:\n EXTI5: S1\n EXTI6: S2\n EXTI7: S3\n EXTI8: S4\n EXTI9:\n\nEXTI15_10:\n EXTI10: \n EXTI11: INT1_A\n EXTI12: INT1_G\n EXTI13: INT2_A\n EXTI14: \n EXTI15: DRDYg/INT2_G"

Commit message: cpld: Added two LEDS and removed the EXTIO0 and EXTI1 since they are already used by the sensor discovery: Rearranged pins to connect both audio lines to adjacent ADCs as well as to free up pins as a result of not using EXTI0 and EXTI1 f4_daughter: Moved around some stuff and changed relevant text
Parts:
- removed S?: EVQ-Q2S03W, symbol EVQ-Q2S03W
- added D? (x2): LED, symbol LED
- added R? (x2): 10k, symbol RES
- added S?: EVQ-Q2S03W, symbol EVQ-Q2S03W
Connections:
- net labels added: LED1, LED2
- net labels removed: EXTI0, EXTI1
- wire segments 113 -> 119

Commit message: Annotated, removed duplicate datasheet and CPLD.sch
Parts:
- removed P?: CONN_5, symbol CONN_5
- added P1: CONN_6, symbol CONN_6
- gave numbers to parts that had none: 9
Connections:
- wire segments 119 -> 121

Commit message: Cleaned up antenna symbols and more footprint associations
Parts:
- renumbered P1 to J2
Changed lines of the file:
@@
-EESchema Schematic File Version 2  date 1/8/2013 5:13:17 PM
+EESchema Schematic File Version 2  date Wed 09 Jan 2013 04:33:42 PM EST
 LIBS:power
 LIBS:device
@@
 Sheet 4 9
 Title ""
-Date "8 jan 2013"
+Date "9 jan 2013"
 Rev ""
 Comp ""
@@
 $EndComp
 $Comp
-L CONN_6 P1
+L CONN_6 J2
 U 1 1 50EAFAC5
 P 5200 6650
-F 0 "P1" V 5150 6650 60  0000 C CNN
+F 0 "J2" V 5150 6650 60  0000 C CNN
 F 1 "CONN_6" V 5250 6650 60  0000 C CNN
 	1    5200 6650

Commit message: Moved around the cpld for easier connections.
Connections:
- wire segments 121 -> 118

Commit message: Almost finished wiring up the CPLD.
Connections:
- wire segments 118 -> 117

Commit message: Fixed a few things: CPLD_EN now a pin on STM32F4 Took FSMC_A16 off of CPLD Put BKLT_EN on the CPLD Rework FTDI chip connections
Connections:
- net labels added: BKLT_EN, POW_nCHRG, V1.8
- net labels removed: FSMC_A16, RS
Changed lines of the file:
@@
-EESchema Schematic File Version 2  date Wed 16 Jan 2013 06:45:33 PM EST
+EESchema Schematic File Version 2  date Thu 17 Jan 2013 02:12:00 PM EST
 LIBS:power
 LIBS:device
@@
 $Descr A4 11700 8267
 encoding utf-8
-Sheet 4 9
+Sheet 5 9
 Title ""
-Date "16 jan 2013"
+Date "17 jan 2013"
 Rev ""
 Comp ""
@@
 Comment4 ""
 $EndDescr
+Text Label 9350 5300 2    60   ~ 0
+POW_nCHRG
+Text HLabel 9650 5300 2    60   Input ~ 0
+POW_nCHRG
+Wire Wire Line
+	9650 5300 9350 5300
+Text Label 4400 3000 2    60   ~ 0
+POW_nCHRG
+Text HLabel 9600 4300 2    60   Output ~ 0
+BKLT_EN
+Text Label 9300 4300 2    60   ~ 0
+BKLT_EN
+Wire Wire Line
+	9600 4300 9300 4300
+Text Label 4400 3100 2    60   ~ 0
+BKLT_EN
 Wire Wire Line
 	6950 2450 6950 2500
@@
 	4550 3000 4400 3000
 Wire Wire Line
-	1900 5050 2150 5050
-Wire Wire Line
 	1900 4750 2150 4750
 Wire Wire Line
@@
 	6250 3700 6250 3850
 Wire Wire Line
-	9600 4300 9300 4300
-Wire Wire Line
 	9600 4100 9300 4100
 Wire Wire Line
@@
 	5750 1250 5700 1250
 $Comp
-L GND #PWR07
+L GND #PWR08
 U 1 1 50EAFAE0
 P 4750 7000
-F 0 "#PWR07" H 4750 7000 30  0001 C CNN
+F 0 "#PWR08" H 4750 7000 30  0001 C CNN
 F 1 "GND" H 4750 6930 30  0001 C CNN
 	1    4750 7000
@@
 $EndComp
 $Comp
-L GND #PWR08
+L GND #PWR09
 U 1 1 50E5F5D9
 P 7750 6250
-F 0 "#PWR08" H 7750 6250 30  0001 C CNN
+F 0 "#PWR09" H 7750 6250 30  0001 C CNN
 F 1 "GND" H 7750 6180 30  0001 C CNN
 	1    7750 6250
@@
 $EndComp
 $Comp
-L GND #PWR09
+L GND #PWR010
 U 1 1 50E5F4E2
 P 7400 5425
-F 0 "#PWR09" H 7400 5425 30  0001 C CNN
+F 0 "#PWR010" H 7400 5425 30  0001 C CNN
 F 1 "GND" H 7400 5355 30  0001 C CNN
 	1    7400 5425
@@
 S1
 $Comp
-L GND #PWR010
+L GND #PWR011
 U 1 1 50D22294
 P 5500 5425
-F 0 "#PWR010" H 5500 5425 30  0001 C CNN
+F 0 "#PWR011" H 5500 5425 30  0001 C CNN
 F 1 "GND" H 5500 5355 30  0001 C CNN
 	1    5500 5425
@@
 $EndComp
 $Comp
-L GND #PWR011
+L GND #PWR012
 U 1 1 50D22293
 P 6500 5425
-F 0 "#PWR011" H 6500 5425 30  0001 C CNN
+F 0 "#PWR012" H 6500 5425 30  0001 C CNN
 F 1 "GND" H 6500 5355 30  0001 C CNN
 	1    6500 5425
@@
 $EndComp
 $Comp
-L GND #PWR012
+L GND #PWR013
 U 1 1 50D22292
 P 4550 5425
-F 0 "#PWR012" H 4550 5425 30  0001 C CNN
+F 0 "#PWR013" H 4550 5425 30  0001 C CNN
 F 1 "GND" H 4550 5355 30  0001 C CNN
 	1    4550 5425
@@
 JTAG Header
 Text GLabel 5850 1250 1    60   Input ~ 0
-Vreg
+V1.8
 Text Label 4400 2300 2    60   ~ 0
 JTDO
@@
 Vreg
 $Comp
-L GND #PWR013
+L GND #PWR014
 U 1 1 50C8FC57
 P 6950 2800
-F 0 "#PWR013" H 6950 2800 30  0001 C CNN
+F 0 "#PWR014" H 6950 2800 30  0001 C CNN
 F 1 "GND" H 6950 2730 30  0001 C CNN
 	1    6950 2800
@@
 Text Label 6950 2700 0    60   ~ 0
 S3
-Text Label 2150 5050 0    60   ~ 0
-FSMC_A16
 Text Label 2150 4900 0    60   ~ 0
 FSMC_NWE
 Text Label 2150 4750 0    60   ~ 0
 FSMC_NEx
-Text HLabel 1900 5050 0    60   Input ~ 0
-FSMC_A16
 Text HLabel 1900 4900 0    60   Input ~ 0
 FSMC_NWE
@@
 FSMC_NEx
 $Comp
-L GND #PWR014
+L GND #PWR015
 U 1 1 50C8F5AA
 P 5650 1350
-F 0 "#PWR014" H 5650 1350 30  0001 C CNN
+F 0 "#PWR015" H 5650 1350 30  0001 C CNN
 F 1 "GND" H 5650 1280 30  0001 C CNN
 	1    5650 1350
@@
 $EndComp
 $Comp
-L GND #PWR015
+L GND #PWR016
 U 1 1 50C8F5A0
 P 4400 2400
-F 0 "#PWR015" H 4400 2400 30  0001 C CNN
+F 0 "#PWR016" H 4400 2400 30  0001 C CNN
 F 1 "GND" H 4400 2330 30  0001 C CNN
 	1    4400 2400
@@
 Text Label 4400 2700 2    60   ~ 0
 EXTI12
-Text Label 4400 3000 2    60   ~ 0
-FSMC_A16
 Text Label 4400 2900 2    60   ~ 0
 nWR
-Text Label 4400 3100 2    60   ~ 0
-RS
 Text Label 5550 3850 3    60   ~ 0
 EXTI6
@@
 Text HLabel 9600 4500 2    60   Input ~ 0
 SPI_SCK
-Text Label 9300 4300 2    60   ~ 0
-RS
 Text Label 9300 4200 2    60   ~ 0
 nWR
@@
 Text Label 9300 3200 2    60   ~ 0
 INT1_ACC
-Text HLabel 9600 4300 2    60   Output ~ 0
-RS
 Text HLabel 9600 4200 2    60   Output ~ 0
 nWR
