File: pcb/lcd.sch (KiCad schematic (older format))
At the start: 1 part, among them J4 ITDB_TFT

Commit message: Added backlight driver, connected to I2C1, annotated stuff
Parts:
- added C44, C45: 10u, symbol CAP
- added L5: CVH252009-1R0M, symbol INDUCTOR
- added R36: 220k, symbol RES
- added R37, R38: 0R, symbol RES
- added U15: LM3561, symbol LM3561
Connections:
- net labels added: BACKLIGHT, BKLT_EN, BKLT_SCL, BKLT_SDA, Vbat
- net labels removed: LCD_BKLIGHT
- wire segments 74 -> 91
