File: pcb/cc3000.sch (KiCad schematic (older format))
At the start: 9 parts, among them P1 CONN_5, U4 CC3000

Commit message: Fixed a line in the schematic file that caused an error message
Connections:
- net labels removed: 
Changed lines of the file:
@@
-EESchema Schematic File Version 2  date 7/22/2013 10:56:01 PM
+EESchema Schematic File Version 2  date 10/27/2013 8:54:36 PM
 LIBS:power
 LIBS:device
@@
 $EndComp
 Text Label 5800 4650 3    60   ~ 0
+SPI_DIN
 Text Label 6000 4650 3    60   ~ 0
 SPI_CLK
